File: Archive/nereus_Pi_shield_ADIN2111_001/BM_Mote_1_Master.kicad_sch (KiCad schematic)
At the start: 50 parts, among them J3 TC2030-FP-sofar, P1 DF17(3.0)-30DS-0.5V(57)

Commit message: updated with fix junctions in the schematic
Parts:
- removed J3: TC2030-FP-sofar, TC2030-FP-Footprint-1, symbol BM_Mote_000639-AB-altium-import:Designator_0_mirrored_TC2030-FP-Symbol-1_Sofar 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
- removed TP25, TP26, TP37: TEST_POINT, PCB_TP_1.5mm, symbol BM_Mote_000639-AB-altium-import:Designator_3_TEST_POINT_Sofar Ocean Technologie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
- removed TP27, TP28, TP30: TEST_POINT, PCB_TP_1.5mm, symbol BM_Mote_000639-AB-altium-import:Designator_2_mirrored_TEST_POINT_Sofar Ocean Te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
- removed TP29: TEST_POINT, PCB_TP_1.5mm, symbol BM_Mote_000639-AB-altium-import:Designator_1_TEST_POINT_Sofar Ocean Technologie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
Connections:
- no-connect marks 4 -> 2
Other:
- removed sheet Processor
- removed sheet USB
