File: nereus_Pi_shield_ADIN2111/BM_Mote_1_Master.kicad_sch (KiCad schematic)
At the start: 33 parts, among them J1 Raspberry_Pi_2_3

Commit message: S5.d: payload connector J5 (JST GH 2-pin SM02B-GHS-TB) on the Top-Level sheet
Pin 1 VBUS_OUT, pin 2 GND (UrchinCam J4/J6 order); 1.0 A/contact, 50 V (JST GH
datasheet). Symbol copied from the UrchinCam into nereus.kicad_sym. Netlist:
VBUS_OUT + J5.1, GND + J5.2 only; ERC 27/508 unchanged; netcheck 51/51. D23.

Co-Authored-By: Claude Opus 5.5 <noreply@anthropic.com>
Parts:
- added J5: SM02B-GHS-TB, Connector_JST:JST_GH_SM02B-GHS-TB_1x02-1MP_P1.25mm_Horizontal, symbol nereus:SM02B-GHS
Connections:
- net GND: now also J5.2 (Pin_2)
- net VBUS_OUT: now also J5.1 (Pin_1)
Other:
- note added: "Payload power out: J5, JST GH 1.25 mm (D23). Pin 1 VBUS_OUT: 16-32 V bus, switched by U11, ~0.73 A limit. Pin 2 GND. Pin order as the UrchinCam J4/J6. Mate the cable before potting."
Changed lines of the file:
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@@
 		)
 	)
+	(text "Payload power out: J5, JST GH 1.25 mm (D23).\nPin 1 VBUS_OUT: 16-32 V bus, switched by U11,\n~0.73 A limit. Pin 2 GND.\nPin order as the UrchinCam J4/J6.\nMate the cable before potting."
+		(exclude_from_sim no)
+		(at 35.56 177.8 0)
+		(effects
+			(font
+				(size 1.27 1.27)
+			)
+			(justify left top)
+		)
+	)
 	(text_box "Processor + onboard logic runs off 3V3, and ADIN AVDD off 1V8."
 		(exclude_from_sim no)
@@
 		)
 	)
+	(wire
+		(pts
+			(xy 66.04 160.02) (xy 50.8 160.02)
+		)
+		(stroke
+			(width 0)
+			(type default)
+		)
+	)
+	(wire
+		(pts
+			(xy 66.04 162.56) (xy 55.88 162.56)
+		)
+		(stroke
+			(width 0)
+			(type default)
+		)
+	)
 	(label "BM2_P"
 		(at 454.66 121.92 0)
@@
 					(unit 1)
 				)
+			)
+		)
+	)
+	(symbol
+		(lib_id "nereus:SM02B-GHS")
+		(at 71.12 161.29 0)
+		(unit 1)
+		(exclude_from_sim no)
+		(in_bom yes)
+		(on_board yes)
+		(dnp no)
+		(property "Reference" "J5"
+			(at 71.12 157.48 0)
+			(effects
+				(font
+					(size 1.27 1.27)
+				)
+			)
+		)
+		(property "Value" "SM02B-GHS-TB"
+			(at 71.12 166.37 0)
+			(effects
+				(font
+					(size 1.27 1.27)
+				)
+			)
+		)
+		(property "Footprint" "Connector_JST:JST_GH_SM02B-GHS-TB_1x02-1MP_P1.25mm_Horizontal"
+			(at 71.12 161.29 0)
+			(effects
+				(font
+					(size 1.27 1.27)
+				)
+				(hide yes)
+			)
+		)
+		(property "Datasheet" "https://www.jst-mfg.com/product/pdf/eng/eGH.pdf"
+			(at 71.12 161.29 0)
+			(effects
+				(font
+					(size 1.27 1.27)
+				)
+				(hide yes)
+			)
+		)
+		(property "Description" "JST GH 1.25 mm 2-pin SMD right-angle header, 1.0 A per contact (AWG #26), 50 V: payload power out, pin 1 VBUS_OUT, pin 2 GND (D23)"
+			(at 71.12 161.29 0)
+			(effects
+				(font
+					(size 1.27 1.27)
+				)
+				(hide yes)
+			)
+		)
+		(property "MANUFACTURER" "JST"
+			(at 71.12 161.29 0)
+			(effects
+				(font
+					(size 1.27 1.27)
+				)
+				(hide yes)
+			)
+		)
+		(property "LCSC" "C189893"
+			(at 71.12 161.29 0)
+			(effects
+				(font
+					(size 1.27 1.27)
+				)
+				(hide yes)
+			)
+		)
+		(pin "1"
+		)
+		(pin "2"
+		)
+		(instances
+			(project ""
+				(path "/30e82bf5-1344-486b-817c-02d3b0649ce4/3c398828-e355-49f6-be37-cb3640d2c671"
+					(reference "J5")
+					(unit 1)
+				)
+			)
+		)
+	)
+	(symbol
+		(lib_id "BM_Mote_000639-AB-altium-import:VBUS_OUT_BAR")
+		(at 50.8 160.02 180)
+		(unit 1)
+		(exclude_from_sim no)
+		(in_bom yes)
+		(on_board yes)
+		(dnp no)
+		(property "Reference" "#PWR80"
+			(at 50.8 156.21 0)
+			(effects
+				(font
+					(size 1.27 1.27)
+				)
+				(hide yes)
+			)
+		)
+		(property "Value" "VBUS_OUT"
+			(at 50.8 156.21 0)
+			(effects
+				(font
+					(size 1.27 1.27)
+				)
+			)
+		)
+		(property "Footprint" ""
+			(at 50.8 160.02 0)
+			(effects
+				(font
+					(size 1.27 1.27)
+				)
+				(hide yes)
+			)
+		)
+		(property "Datasheet" ""
+			(at 50.8 160.02 0)
+			(effects
+				(font
+					(size 1.27 1.27)
+				)
+				(hide yes)
+			)
+		)
+		(property "Description" ""
+			(at 50.8 160.02 0)
+			(effects
+				(font
+					(size 1.27 1.27)
+				)
+				(hide yes)
+			)
+		)
+		(pin ""
+		)
+		(instances
+			(project ""
+				(path "/30e82bf5-1344-486b-817c-02d3b0649ce4/3c398828-e355-49f6-be37-cb3640d2c671"
+					(reference "#PWR80")
+					(unit 1)
+				)
+			)
+		)
+	)
+	(symbol
+		(lib_id "BM_Mote_000639-AB-altium-import:GND_POWER_GROUND")
+		(at 55.88 162.56 0)
+		(unit 1)
+		(exclude_from_sim no)
+		(in_bom yes)
+		(on_board yes)
+		(dnp no)
+		(property "Reference" "#PWR81"
+			(at 55.88 158.75 0)
+			(effects
+				(font
+					(size 1.27 1.27)
+				)
+				(hide yes)
+			)
+		)
+		(property "Value" "GND"
+			(at 55.88 170.18 0)
+			(effects
+				(font
+					(size 1.27 1.27)
+				)
+			)
+		)
+		(property "Footprint" ""
+			(at 55.88 162.56 0)
+			(effects
+				(font
+					(size 1.27 1.27)
+				)
+				(hide yes)
+			)
+		)
+		(property "Datasheet" ""
+			(at 55.88 162.56 0)
+			(effects
+				(font
+					(size 1.27 1.27)
+				)
+				(hide yes)
+			)
+		)
+		(property "Description" ""
+			(at 55.88 162.56 0)
+			(effects
+				(font
+					(size 1.27 1.27)
+				)
+				(hide yes)
+			)
+		)
+		(pin ""
+		)
+		(instances
+			(project ""
+				(path "/30e82bf5-1344-486b-817c-02d3b0649ce4/3c398828-e355-49f6-be37-cb3640d2c671"
+					(reference "#PWR81")
+					(unit 1)
+				)

Commit message: S5.d: J5 moved to the right side under the PoDL inserts (interconnects live there); note without the UrchinCam ref; Molex bus note -> M3 threaded inserts; S6 tidy item
Netlist identical to before the move; ERC 27/508; netcheck 51/51.

Co-Authored-By: Claude Opus 5.5 <noreply@anthropic.com>
Other:
- note added: "Payload power out: J5, JST GH 1.25 mm (D23). Pin 1 VBUS_OUT: 16-32 V bus, switched by U11, ~0.73 A limit. Pin 2 GND. Mate the cable before potting."
- note removed: "Payload power out: J5, JST GH 1.25 mm (D23). Pin 1 VBUS_OUT: 16-32 V bus, switched by U11, ~0.73 A limit. Pin 2 GND. Pin order as the UrchinCam J4/J6. Mate the cable before potting."
- moved on the sheet: J5
Changed lines of the file:
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@@
 		)
 	)
-	(text "Payload power out: J5, JST GH 1.25 mm (D23).\nPin 1 VBUS_OUT: 16-32 V bus, switched by U11,\n~0.73 A limit. Pin 2 GND.\nPin order as the UrchinCam J4/J6.\nMate the cable before potting."
+	(text "Payload power out: J5, JST GH 1.25 mm (D23).\nPin 1 VBUS_OUT: 16-32 V bus, switched by U11,\n~0.73 A limit. Pin 2 GND.\nMate the cable before potting."
 		(exclude_from_sim no)
-		(at 35.56 177.8 0)
+		(at 454.66 177.8 0)
 		(effects
 			(font
@@
 		)
 	)
-	(text_box "Bristlemouth Bus:\nMolex 2-pin"
+	(text_box "Bristlemouth bus:\nM3 threaded inserts\nMP1-MP4"
 		(exclude_from_sim no)
 		(at 481.33 133.35 0)
-		(size -29.21 13.97)
+		(size -29.21 19.05)
 		(margins 0.9525 0.9525 0.9525 0.9525)
 		(stroke
@@
 	(wire
 		(pts
-			(xy 66.04 160.02) (xy 50.8 160.02)
+			(xy 485.14 160.02) (xy 469.9 160.02)
 		)
 		(stroke
@@
 	(wire
 		(pts
-			(xy 66.04 162.56) (xy 55.88 162.56)
+			(xy 485.14 162.56) (xy 474.98 162.56)
 		)
 		(stroke
@@
 	(symbol
 		(lib_id "nereus:SM02B-GHS")
-		(at 71.12 161.29 0)
+		(at 490.22 161.29 0)
 		(unit 1)
 		(exclude_from_sim no)
@@
 		(dnp no)
 		(property "Reference" "J5"
-			(at 71.12 157.48 0)
+			(at 490.22 157.48 0)
 			(effects
 				(font
@@
 		)
 		(property "Value" "SM02B-GHS-TB"
-			(at 71.12 166.37 0)
+			(at 490.22 166.37 0)
 			(effects
 				(font
@@
 		)
 		(property "Footprint" "Connector_JST:JST_GH_SM02B-GHS-TB_1x02-1MP_P1.25mm_Horizontal"
-			(at 71.12 161.29 0)
+			(at 490.22 161.29 0)
 			(effects
 				(font
@@
 		)
 		(property "Datasheet" "https://www.jst-mfg.com/product/pdf/eng/eGH.pdf"
-			(at 71.12 161.29 0)
+			(at 490.22 161.29 0)
 			(effects
 				(font
@@
 		)
 		(property "Description" "JST GH 1.25 mm 2-pin SMD right-angle header, 1.0 A per contact (AWG #26), 50 V: payload power out, pin 1 VBUS_OUT, pin 2 GND (D23)"
-			(at 71.12 161.29 0)
+			(at 490.22 161.29 0)
 			(effects
 				(font
@@
 		)
 		(property "MANUFACTURER" "JST"
-			(at 71.12 161.29 0)
+			(at 490.22 161.29 0)
 			(effects
 				(font
@@
 		)
 		(property "LCSC" "C189893"
-			(at 71.12 161.29 0)
+			(at 490.22 161.29 0)
 			(effects
 				(font
@@
 	(symbol
 		(lib_id "BM_Mote_000639-AB-altium-import:VBUS_OUT_BAR")
-		(at 50.8 160.02 180)
+		(at 469.9 160.02 180)
 		(unit 1)
 		(exclude_from_sim no)
@@
 		(dnp no)
 		(property "Reference" "#PWR80"
-			(at 50.8 156.21 0)
+			(at 469.9 156.21 0)
 			(effects
 				(font
@@
 		)
 		(property "Value" "VBUS_OUT"
-			(at 50.8 156.21 0)
+			(at 469.9 156.21 0)
 			(effects
 				(font
@@
 		)
 		(property "Footprint" ""
-			(at 50.8 160.02 0)
+			(at 469.9 160.02 0)
 			(effects
 				(font
@@
 		)
 		(property "Datasheet" ""
-			(at 50.8 160.02 0)
+			(at 469.9 160.02 0)
 			(effects
 				(font
@@
 		)
 		(property "Description" ""
-			(at 50.8 160.02 0)
+			(at 469.9 160.02 0)
 			(effects
 				(font
@@
 	(symbol
 		(lib_id "BM_Mote_000639-AB-altium-import:GND_POWER_GROUND")
-		(at 55.88 162.56 0)
+		(at 474.98 162.56 0)
 		(unit 1)
 		(exclude_from_sim no)
@@
 		(dnp no)
 		(property "Reference" "#PWR81"
-			(at 55.88 158.75 0)
+			(at 474.98 158.75 0)
 			(effects
 				(font
@@
 		)
 		(property "Value" "GND"
-			(at 55.88 170.18 0)
+			(at 474.98 170.18 0)
 			(effects
 				(font
@@
 		)
 		(property "Footprint" ""
-			(at 55.88 162.56 0)
+			(at 474.98 162.56 0)
 			(effects
 				(font
@@
 		)
 		(property "Datasheet" ""
-			(at 55.88 162.56 0)
+			(at 474.98 162.56 0)
 			(effects
 				(font
@@
 		)
 		(property "Description" ""
-			(at 55.88 162.56 0)
+			(at 474.98 162.56 0)
 			(effects
 				(font

Commit message: S5.h: BOM alternates as hidden ALT/SOURCING fields; tracked bom.csv
- 24 flagged passives: hidden ALT1/ALT2 MPN/MFR/LCSC, ALT NOTE, SOURCING
  (values from docs/design-review/bom_alternates.md, D26)
- Critical parts (U1-U3, L3/L6, Y1, D1-D3, MP1-MP4, J5, J1): SOURCING only
- tools/check.sh exports docs/design-review/bom.csv: specified part first,
  alternates beside it; grouped by Value + DNP (R11 apart from R12/R13/R17/R19)
- J1 Footprint property re-indented (whitespace; import leftover)
- Fields only: ERC 531/27/504 unchanged, netcheck 51/51, midwire 0;
  netlist diff = the 208 new fields
- Docs: bom_alternates, bom_lifecycle, sofar_brief, changelog, DESIGN,
  TRACKER, viewer, DEV_LOG

Co-Authored-By: Claude Opus 5.5 <noreply@anthropic.com>
Parts:
- J1: SOURCING (none) -> Part not chosen: 2x20 2.54 mm female TH socket, height open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
- J5: SOURCING (none) -> JLC global sourcing (D26); LCSC C189893 out of stock, DK 10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
- MP1, MP2, MP3, MP4: SOURCING (none) -> JLC global sourcing (D26); no LCSC listing, DK 7,835
- R43: ALT NOTE (none) -> 100 kΩ ±1 % 62.5 mW 50 V ±100 ppm; ALT1 is JLC Basic; AEC-Q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; ALT1 LCSC (none) -> C25741; ALT1 MFR (none) -> UNI-ROYAL; ALT1 MPN (none) -> 0402WGF1003TCE; ALT2 LCSC (none) -> C60491; ALT2 MFR (none) -> YAGEO; ALT2 MPN (none) -> RC0402FR-07100KL; SOURCING (none) -> JLC global sourcing (first build) until an ALT is approved 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
Changed lines of the file:
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@@
 			)
 		)
+		(property "SOURCING" "JLC global sourcing (D26); no LCSC listing, DK 7,835"
+			(at 485.14 121.92 0)
+			(effects
+				(font
+					(size 1.27 1.27)
+				)
+				(hide yes)
+			)
+		)
 		(pin "1"
 		)
@@
 			)
 		)
+		(property "SOURCING" "JLC global sourcing (D26); no LCSC listing, DK 7,835"
+			(at 485.14 137.16 0)
+			(effects
+				(font
+					(size 1.27 1.27)
+				)
+				(hide yes)
+			)
+		)
 		(pin "1"
 		)
@@
 			)
 		)
+		(property "SOURCING" "JLC global sourcing (D26); no LCSC listing, DK 7,835"
+			(at 485.14 106.68 0)
+			(effects
+				(font
+					(size 1.27 1.27)
+				)
+				(hide yes)
+			)
+		)
 		(pin "1"
 		)
@@
 			)
 		)
+		(property "SOURCING" "JLC global sourcing (D26); no LCSC listing, DK 7,835"
+			(at 485.14 91.44 0)
+			(effects
+				(font
+					(size 1.27 1.27)
+				)
+				(hide yes)
+			)
+		)
 		(pin "1"
 		)
@@
 			)
 		)
-				(property "Footprint" "Connector_PinSocket_2.54mm:PinSocket_2x20_P2.54mm_Vertical"
+		(property "Footprint" "Connector_PinSocket_2.54mm:PinSocket_2x20_P2.54mm_Vertical"
 			(at 121.92 88.9 0)
 			(effects
@@
 			)
 		)
+		(property "SOURCING" "Part not chosen: 2x20 2.54 mm female TH socket, height open (Nick). Candidates ZHOURI 2.54-2*20 C2977589, Megastar ZX-PM2.54-2-20PY C7499354 (both 8.5 mm)"
+			(at 121.92 88.9 0)
+			(effects
+				(font
+					(size 1.27 1.27)
+				)
+				(hide yes)
+			)
+		)
 		(pin "8"
 		)
@@
 			)
 		)
+		(property "ALT1 MPN" "0402WGF1003TCE"
+			(at 78.74 99.06 0)
+			(effects
+				(font
+					(size 1.27 1.27)
+				)
+				(hide yes)
+			)
+		)
+		(property "ALT1 MFR" "UNI-ROYAL"
+			(at 78.74 99.06 0)
+			(effects
+				(font
+					(size 1.27 1.27)
+				)
+				(hide yes)
+			)
+		)
+		(property "ALT1 LCSC" "C25741"
+			(at 78.74 99.06 0)
+			(effects
+				(font
+					(size 1.27 1.27)
+				)
+				(hide yes)
+			)
+		)
+		(property "ALT2 MPN" "RC0402FR-07100KL"
+			(at 78.74 99.06 0)
+			(effects
+				(font
+					(size 1.27 1.27)
+				)
+				(hide yes)
+			)
+		)
+		(property "ALT2 MFR" "YAGEO"
+			(at 78.74 99.06 0)
+			(effects
+				(font
+					(size 1.27 1.27)
+				)
+				(hide yes)
+			)
+		)
+		(property "ALT2 LCSC" "C60491"
+			(at 78.74 99.06 0)
+			(effects
+				(font
+					(size 1.27 1.27)
+				)
+				(hide yes)
+			)
+		)
+		(property "ALT NOTE" "100 kΩ ±1 % 62.5 mW 50 V ±100 ppm; ALT1 is JLC Basic; AEC-Q200 not stated (Stackpole is)"
+			(at 78.74 99.06 0)
+			(effects
+				(font
+					(size 1.27 1.27)
+				)
+				(hide yes)
+			)
+		)
+		(property "SOURCING" "JLC global sourcing (first build) until an ALT is approved (D26)"
+			(at 78.74 99.06 0)
+			(effects
+				(font
+					(size 1.27 1.27)
+				)
+				(hide yes)
+			)
+		)
 		(pin "2"
 		)
@@
 			(at 490.22 161.29 0)
 			(effects
+				(font
+					(size 1.27 1.27)
+				)
+				(hide yes)
+			)
+		)
+		(property "SOURCING" "JLC global sourcing (D26); LCSC C189893 out of stock, DK 10,839"
+			(at 490.22 161.29 0)
+			(effects

Commit message: S5.h: QE round 1 APPROVED WITH NITS -- nits fixed; alternates capped at 3
- R8 ALT NOTE shortened (Nick: at most 3 alternates per part; R8's 7 Sofar
  fields stay untouched, outside bom.csv)
- J1 SOURCING back to the plan's "2x20" with the multiplication sign (N1);
  C22/C23 DK-figure drop declared in the changelog (N1)
- S6 item: TP/FID/MTG rows in bom.csv for a JLC order (N2)
- QE report recorded in docs/design-review/qe/S5.md; TRACKER, viewer, DEV_LOG

Co-Authored-By: Claude Opus 5.5 <noreply@anthropic.com>
Parts:
- J1: SOURCING Part not chosen: 2x20 2.54 mm female TH socket, height open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 -> Part not chosen: 2×20 2.54 mm female TH socket, height open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
Changed lines of the file:
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@@
 			)
 		)
-		(property "SOURCING" "Part not chosen: 2x20 2.54 mm female TH socket, height open (Nick). Candidates ZHOURI 2.54-2*20 C2977589, Megastar ZX-PM2.54-2-20PY C7499354 (both 8.5 mm)"
+		(property "SOURCING" "Part not chosen: 2×20 2.54 mm female TH socket, height open (Nick). Candidates ZHOURI 2.54-2*20 C2977589, Megastar ZX-PM2.54-2-20PY C7499354 (both 8.5 mm)"
 			(at 121.92 88.9 0)
 			(effects

Commit message: S5.i: planned part per BOM line (D27) beside Sofar's specified part
- PLANNED MPN/MFR/LCSC + PLANNED NOTE (why) on all 106 purchased parts;
  Value (Sofar's part) unchanged
- 10 lines planned as LCSC-stocked equivalents (R34, R20/R39, R21 group,
  C31, C17/C26, C21, C16 group, C19/C27, R14/R18) and D1 -> Sofar's Vishay
  second source; R8 kept (no ROHM land pattern); J1 TBD; rest as specified
- SOURCING on the 19 changed-line parts: planned part after Sofar approves
- Footprint lines of U11, R41, C56-C58 re-indented (whitespace only)
- View "Sofar review (planned parts)"; check.sh exports bom.csv from it
- Fields only: ERC 531/27/504 unchanged, netcheck 51/51, midwire 0
- Docs: DESIGN D27, bom_alternates, bom_lifecycle, sofar_brief, changelog,
  TRACKER, viewer, DEV_LOG

Co-Authored-By: Claude Opus 5.5 <noreply@anthropic.com>
Parts:
- J1: PLANNED MPN (none) -> TBD; PLANNED NOTE (none) -> Part not chosen: 2×20 2.54 mm female TH socket, height open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
- J5: PLANNED LCSC (none) -> C189893; PLANNED MFR (none) -> JST; PLANNED MPN (none) -> SM02B-GHS-TB; PLANNED NOTE (none) -> As specified; LCSC listing out of stock (2026-10-06): JLC g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
- MP1, MP2, MP3, MP4: PLANNED MFR (none) -> Würth Elektronik; PLANNED MPN (none) -> 78614015360; PLANNED NOTE (none) -> As specified; JLC global sourcing (D26): no LCSC listing
- R11: PLANNED LCSC (none) -> C844880; PLANNED MFR (none) -> Vishay Dale; PLANNED MPN (none) -> CRCW12100000Z0EA; PLANNED NOTE (none) -> As specified; DNP (not fitted)
- R26, R27: PLANNED LCSC (none) -> C400631; PLANNED MFR (none) -> Panasonic; PLANNED MPN (none) -> ERJ-2RKF4701X; PLANNED NOTE (none) -> As specified; in LCSC stock (checked 2026-10-06)
- R43: PLANNED LCSC (none) -> C25741; PLANNED MFR (none) -> UNI-ROYAL; PLANNED MPN (none) -> 0402WGF1003TCE; PLANNED NOTE (none) -> JLC Basic part (no extended-part fee), largest LCSC stock; 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; SOURCING JLC global sourcing (first build) until an ALT is approved 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 -> Planned part from LCSC once Sofar approves it (D27); until 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

Commit message: S5.i: QE round 1 APPROVED WITH NITS -- notes fixed; record report; S5 complete
- F1: R21 group "ample LCSC stock"; C16 group stock figures stated
- N1: C17/C26 note no longer claims the same part (thickness not confirmed)
- N2: D26 marked "amended by D27"; N3: C21 note reworded
- R8 datasheet URLs in bom_alternates.md
- QE report in docs/design-review/qe/S5.md; TRACKER, viewer, DEV_LOG

Co-Authored-By: Claude Opus 5.5 <noreply@anthropic.com>
Parts:
- R43: PLANNED NOTE JLC Basic part (no extended-part fee), largest LCSC stock; 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 -> JLC Basic part (no extended-part fee), ample LCSC stock; 10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
Changed lines of the file:
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@@
 			)
 		)
-		(property "PLANNED NOTE" "JLC Basic part (no extended-part fee), largest LCSC stock; 100 kΩ ±1 % 62.5 mW 50 V ±100 ppm 0402; specified Stackpole is out of stock at LCSC and is AEC-Q200, this one doesn't state it"
+		(property "PLANNED NOTE" "JLC Basic part (no extended-part fee), ample LCSC stock; 100 kΩ ±1 % 62.5 mW 50 V ±100 ppm 0402; specified Stackpole is out of stock at LCSC and is AEC-Q200, this one doesn't state it"
 			(at 78.74 99.06 0)
 			(effects

Commit message: S6.a: BOM hygiene -- TP/FID/MTG out of the BOM; MANUFACTURER filled
- in_bom no on TP x16, FID1-6, MTG1-4 (bare copper / holes)
- MANUFACTURER on the 75 BOM parts without one, from bom_lifecycle.md;
  Sofar's MFR_NAME / MANUFACTURER1 / MANUFACTURER 1 untouched; J1 open
- bom.csv 51 rows, Mfr on every row but J1
- ERC 531/27/504 unchanged, netcheck 51/51, midwire 0
- Docs: bom_lifecycle, changelog, DESIGN, TRACKER (S6 bites), viewer, DEV_LOG

Co-Authored-By: Claude Opus 5.5 <noreply@anthropic.com>
Parts:
- FID1, FID2, FID3, FID4, FID5, FID6, MTG1, MTG2, MTG3, MTG4, TP13, TP19, TP20, TP21, TP22, TP23, TP24, TP3, TP36, TP38, TP5, TP7, TP8: now left out of the parts list
- R11: MANUFACTURER (none) -> Vishay Dale
- R26, R27: MANUFACTURER (none) -> Panasonic
- R43: MANUFACTURER (none) -> Stackpole
Changed lines of the file:
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@@
 		(unit 0)
 		(exclude_from_sim no)
-		(in_bom yes)
+		(in_bom no)
 		(on_board yes)
 		(dnp no)
@@
 		(unit 0)
 		(exclude_from_sim no)
-		(in_bom yes)
+		(in_bom no)
 		(on_board yes)
 		(dnp no)
@@
 		(unit 0)
 		(exclude_from_sim no)
-		(in_bom yes)
+		(in_bom no)
 		(on_board yes)
 		(dnp no)
@@
 		(unit 0)
 		(exclude_from_sim no)
-		(in_bom yes)
+		(in_bom no)
 		(on_board yes)
 		(dnp no)
@@
 		(unit 0)
 		(exclude_from_sim no)
-		(in_bom yes)
+		(in_bom no)
 		(on_board yes)
 		(dnp no)
@@
 		(unit 0)
 		(exclude_from_sim no)
-		(in_bom yes)
+		(in_bom no)
 		(on_board yes)
 		(dnp no)
@@
 		(unit 0)
 		(exclude_from_sim no)
-		(in_bom yes)
+		(in_bom no)
 		(on_board yes)
 		(dnp no)
@@
 			)
 		)
+		(property "MANUFACTURER" "Vishay Dale"
+			(at 172.72 190.5 0)
+			(effects
+				(font
+					(size 1.27 1.27)
+				)
+				(hide yes)
+			)
+		)
 		(pin "1"
 		)
@@
 		(unit 0)
 		(exclude_from_sim no)
-		(in_bom yes)
+		(in_bom no)
 		(on_board yes)
 		(dnp no)
@@
 		(unit 0)
 		(exclude_from_sim no)
-		(in_bom yes)
+		(in_bom no)
 		(on_board yes)
 		(dnp no)
@@
 		(unit 0)
 		(exclude_from_sim no)
-		(in_bom yes)
+		(in_bom no)
 		(on_board yes)
 		(dnp no)
@@
 		(unit 0)
 		(exclude_from_sim no)
-		(in_bom yes)
+		(in_bom no)
 		(on_board yes)
 		(dnp no)
@@
 		(unit 0)
 		(exclude_from_sim no)
-		(in_bom yes)
+		(in_bom no)
 		(on_board yes)
 		(dnp no)
@@
 		(unit 0)
 		(exclude_from_sim no)
-		(in_bom yes)
+		(in_bom no)
 		(on_board yes)
 		(dnp no)
@@
 		(unit 0)
 		(exclude_from_sim no)
-		(in_bom yes)
+		(in_bom no)
 		(on_board yes)
 		(dnp no)
@@
 		(unit 0)
 		(exclude_from_sim no)
-		(in_bom yes)
+		(in_bom no)
 		(on_board yes)
 		(dnp no)
@@
 		(unit 0)
 		(exclude_from_sim no)
-		(in_bom yes)
+		(in_bom no)
 		(on_board yes)
 		(dnp no)
@@
 		(unit 0)
 		(exclude_from_sim no)
-		(in_bom yes)
+		(in_bom no)
 		(on_board yes)
 		(dnp no)
@@
 		(unit 0)
 		(exclude_from_sim no)
-		(in_bom yes)
+		(in_bom no)
 		(on_board yes)
 		(dnp no)
@@
 		(unit 0)
 		(exclude_from_sim no)
-		(in_bom yes)
+		(in_bom no)
 		(on_board yes)
 		(dnp no)
@@
 		(unit 0)
 		(exclude_from_sim no)
-		(in_bom yes)
+		(in_bom no)
 		(on_board yes)
 		(dnp no)
@@
 		(unit 0)
 		(exclude_from_sim no)
-		(in_bom yes)
+		(in_bom no)
 		(on_board yes)
 		(dnp no)
@@
 		(unit 0)
 		(exclude_from_sim no)
-		(in_bom yes)
+		(in_bom no)
 		(on_board yes)
 		(dnp no)
@@
 		(unit 0)
 		(exclude_from_sim no)
-		(in_bom yes)
+		(in_bom no)
 		(on_board yes)
 		(dnp no)
@@
 			)
 		)
+		(property "MANUFACTURER" "Panasonic"
+			(at 170.18 60.96 0)
+			(effects
+				(font
+					(size 1.27 1.27)
+				)
+				(hide yes)
+			)
+		)
 		(pin "2"
 		)
@@
 			)
 		)
+		(property "MANUFACTURER" "Panasonic"
+			(at 170.18 66.04 0)
+			(effects
+				(font
+					(size 1.27 1.27)
+				)
+				(hide yes)
+			)
+		)
 		(pin "2"
 		)
@@
 			(at 78.74 99.06 0)
 			(effects
+				(font
+					(size 1.27 1.27)
+				)
+				(hide yes)
+			)
+		)
+		(property "MANUFACTURER" "Stackpole"
+			(at 78.74 99.06 0)
+			(effects
