File: nereus_Pi_shield_ADIN2111/BM_Mote_1_PoDL.kicad_sch (KiCad schematic)
At the start: 28 parts, among them T1 74930000, T2 74930000

Commit message: S4.d: footprints findable -- project library Vault (mote.pretty) extracted from the mote board; close S5.a
43 footprints the schematic uses, extracted read-only from the reference
board with KiCad 9.0.6 pcbnew (tools/fpextract.py, back-side parts
flipped, nets cleared), registered as nickname Vault to match the board
IDs; 118 bare footprint fields -> Vault:<name>. fpextract --verify: 0
problems (negative-tested). Netlist identical except footprint fields.
ERC 74/626 -> 74/508 (footprint-link warnings gone). D19.

Co-Authored-By: Claude Opus 5.5 <noreply@anthropic.com>
Parts:
- C16, C18, C24, C25: footprint FP-0805-L_2_01_0_2-W_1_25-MFG -> Vault:FP-0805-L_2_01_0_2-W_1_25-MFG
- C17, C26: footprint FP-C2012-125-0_2-MFG -> Vault:FP-C2012-125-0_2-MFG
- C19, C27: footprint CAPC2013X145X50LL20T25 -> Vault:CAPC2013X145X50LL20T25
- C20: footprint FP-GRM188-0_1-e0_2_0_5-IPC_B -> Vault:FP-GRM188-0_1-e0_2_0_5-IPC_B
- C21: footprint FP-CL32-IPC_C -> Vault:FP-CL32-IPC_C
- C22, C23: footprint FP-FTD-MFG -> Vault:FP-FTD-MFG
- D1: footprint SMA6F33A-Footprint-1 -> Vault:SMA6F33A-Footprint-1
- D2: footprint FP-PMDTM-MFG -> Vault:FP-PMDTM-MFG
- D4, D5: footprint FP-SOD-323-MFG -> Vault:FP-SOD-323-MFG
- L1, L2: footprint SRF1260-101M-Footprint-1 -> Vault:SRF1260-101M-Footprint-1
- R12, R13, R17, R19: footprint FP-CRCW1210-e3-IPC_B -> Vault:FP-CRCW1210-e3-IPC_B
- R14, R18: footprint FP-RR0510-IPC_B -> Vault:FP-RR0510-IPC_B
- R15, R16: footprint CRCW08057R50FKEAHP-Footprint-1 -> Vault:CRCW08057R50FKEAHP-Footprint-1
- T1, T2: footprint FP-74930000-MFG -> Vault:FP-74930000-MFG
Changed lines of the file:
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@@
 			)
 		)
-		(property "Footprint" ""
+				(property "Footprint" ""
 			(at 116.84 134.4422 0)
 			(effects
@@
 			)
 		)
-		(property "Footprint" "SRF1260-101M-Footprint-1"
+		(property "Footprint" "Vault:SRF1260-101M-Footprint-1"
 			(at 238.76 223.3422 0)
 			(effects
@@
 			)
 		)
-		(property "Footprint" "FP-0805-L_2_01_0_2-W_1_25-MFG"
+		(property "Footprint" "Vault:FP-0805-L_2_01_0_2-W_1_25-MFG"
 			(at 60.96 192.8622 0)
 			(effects
@@
 			)
 		)
-		(property "Footprint" "CRCW08057R50FKEAHP-Footprint-1"
+		(property "Footprint" "Vault:CRCW08057R50FKEAHP-Footprint-1"
 			(at 335.28 134.4422 0)
 			(effects
@@
 			)
 		)
-		(property "Footprint" ""
+				(property "Footprint" ""
 			(at 195.58 246.2022 0)
 			(effects
@@
 			)
 		)
-		(property "Footprint" ""
+				(property "Footprint" ""
 			(at 116.84 246.2022 0)
 			(effects
@@
 			)
 		)
-		(property "Footprint" "FP-SOD-323-MFG"
+		(property "Footprint" "Vault:FP-SOD-323-MFG"
 			(at 43.18 175.0822 0)
 			(effects
@@
 			)
 		)
-		(property "Footprint" "FP-CRCW1210-e3-IPC_B"
+		(property "Footprint" "Vault:FP-CRCW1210-e3-IPC_B"
 			(at 256.54 103.9622 0)
 			(effects
@@
 			)
 		)
-		(property "Footprint" ""
+				(property "Footprint" ""
 			(at 60.96 134.4422 0)
 			(effects
@@
 			)
 		)
-		(property "Footprint" "FP-RR0510-IPC_B"
+		(property "Footprint" "Vault:FP-RR0510-IPC_B"
 			(at 60.96 103.9622 0)
 			(effects
@@
 			)
 		)
-		(property "Footprint" "FP-0805-L_2_01_0_2-W_1_25-MFG"
+		(property "Footprint" "Vault:FP-0805-L_2_01_0_2-W_1_25-MFG"
 			(at 116.84 116.6622 0)
 			(effects
@@
 			)
 		)
-		(property "Footprint" "FP-74930000-MFG"
+		(property "Footprint" "Vault:FP-74930000-MFG"
 			(at 101.6 70.9422 0)
 			(effects
@@
 			)
 		)
-		(property "Footprint" "FP-FTD-MFG"
+		(property "Footprint" "Vault:FP-FTD-MFG"
 			(at 312.42 147.1422 0)
 			(effects
@@
 			)
 		)
-		(property "Footprint" "FP-0805-L_2_01_0_2-W_1_25-MFG"
+		(property "Footprint" "Vault:FP-0805-L_2_01_0_2-W_1_25-MFG"
 			(at 116.84 228.4222 0)
 			(effects
@@
 			)
 		)
-		(property "Footprint" ""
+				(property "Footprint" ""
 			(at 60.96 246.2022 0)
 			(effects
@@
 			)
 		)
-		(property "Footprint" "FP-CRCW1210-e3-IPC_B"
+		(property "Footprint" "Vault:FP-CRCW1210-e3-IPC_B"
 			(at 256.54 73.4822 0)
 			(effects
@@
 			)
 		)
-		(property "Footprint" "FP-CRCW1210-e3-IPC_B"
+		(property "Footprint" "Vault:FP-CRCW1210-e3-IPC_B"
 			(at 256.54 208.1022 0)
 			(effects
@@
 			)
 		)
-		(property "Footprint" "FP-GRM188-0_1-e0_2_0_5-IPC_B"
+		(property "Footprint" "Vault:FP-GRM188-0_1-e0_2_0_5-IPC_B"
 			(at 287.02 142.0622 0)
 			(effects
@@
 			)
 		)
-		(property "Footprint" "CAPC2013X145X50LL20T25"
+		(property "Footprint" "Vault:CAPC2013X145X50LL20T25"
 			(at 58.42 241.1222 0)
 			(effects
@@
 			)
 		)
-		(property "Footprint" "CRCW08057R50FKEAHP-Footprint-1"
+		(property "Footprint" "Vault:CRCW08057R50FKEAHP-Footprint-1"
 			(at 312.42 134.4422 0)
 			(effects
@@
 			)
 		)
-		(property "Footprint" "FP-C2012-125-0_2-MFG"
+		(property "Footprint" "Vault:FP-C2012-125-0_2-MFG"
 			(at 203.2 228.4222 0)
 			(effects
@@
 			)
 		)
-		(property "Footprint" "FP-CL32-IPC_C"
+		(property "Footprint" "Vault:FP-CL32-IPC_C"
 			(at 299.72 142.0622 0)
 			(effects
@@
 			)
 		)
-		(property "Footprint" "FP-0805-L_2_01_0_2-W_1_25-MFG"
+		(property "Footprint" "Vault:FP-0805-L_2_01_0_2-W_1_25-MFG"
 			(at 60.96 81.1022 0)
 			(effects
@@
 			)
 		)
-		(property "Footprint" ""
+				(property "Footprint" ""
 			(at 335.28 159.8422 0)
 			(effects
@@
 			)
 		)
-		(property "Footprint" "FP-C2012-125-0_2-MFG"
+		(property "Footprint" "Vault:FP-C2012-125-0_2-MFG"
 			(at 208.28 93.8022 0)
 			(effects
@@
 			)
 		)
-		(property "Footprint" "FP-RR0510-IPC_B"
+		(property "Footprint" "Vault:FP-RR0510-IPC_B"
 			(at 60.96 215.7222 0)
 			(effects
@@
 			)
 		)
-		(property "Footprint" "FP-PMDTM-MFG"
+		(property "Footprint" "Vault:FP-PMDTM-MFG"
 			(at 383.54 152.2222 0)
 			(effects
@@
 			)
 		)
-		(property "Footprint" "FP-CRCW1210-e3-IPC_B"
+		(property "Footprint" "Vault:FP-CRCW1210-e3-IPC_B"
 			(at 256.54 238.5822 0)
 			(effects
@@
 			)
 		)
-		(property "Footprint" "CAPC2013X145X50LL20T25"
+		(property "Footprint" "Vault:CAPC2013X145X50LL20T25"
 			(at 58.42 129.3622 0)
 			(effects
@@
 			)
 		)
-		(property "Footprint" "FP-SOD-323-MFG"
+		(property "Footprint" "Vault:FP-SOD-323-MFG"
 			(at 43.18 63.3222 0)
 			(effects
@@
 			)
 		)
-		(property "Footprint" "FP-74930000-MFG"
+		(property "Footprint" "Vault:FP-74930000-MFG"
 			(at 101.6 182.7022 0)
 			(effects
@@
 			)
 		)
-		(property "Footprint" "FP-FTD-MFG"
+		(property "Footprint" "Vault:FP-FTD-MFG"
 			(at 335.28 147.1422 0)
 			(effects
@@
 			)
 		)
-		(property "Footprint" "SMA6F33A-Footprint-1"
+		(property "Footprint" "Vault:SMA6F33A-Footprint-1"
 			(at 358.14 144.6022 0)
 			(effects
@@
 			)
 		)
-		(property "Footprint" ""
+				(property "Footprint" ""
 			(at 208.28 111.5822 0)
 			(effects
@@
 			)
 		)
-		(property "Footprint" "SRF1260-101M-Footprint-1"
+		(property "Footprint" "Vault:SRF1260-101M-Footprint-1"
 			(at 238.76 88.7222 0)
 			(effects

Commit message: S5.h: BOM alternates as hidden ALT/SOURCING fields; tracked bom.csv
- 24 flagged passives: hidden ALT1/ALT2 MPN/MFR/LCSC, ALT NOTE, SOURCING
  (values from docs/design-review/bom_alternates.md, D26)
- Critical parts (U1-U3, L3/L6, Y1, D1-D3, MP1-MP4, J5, J1): SOURCING only
- tools/check.sh exports docs/design-review/bom.csv: specified part first,
  alternates beside it; grouped by Value + DNP (R11 apart from R12/R13/R17/R19)
- J1 Footprint property re-indented (whitespace; import leftover)
- Fields only: ERC 531/27/504 unchanged, netcheck 51/51, midwire 0;
  netlist diff = the 208 new fields
- Docs: bom_alternates, bom_lifecycle, sofar_brief, changelog, DESIGN,
  TRACKER, viewer, DEV_LOG

Co-Authored-By: Claude Opus 5.5 <noreply@anthropic.com>
Parts:
- C16, C18, C24, C25: ALT NOTE (none) -> 470 nF ±10 % 100 V X7R 0805; PoDL front end: Sofar review; ALT1 LCSC (none) -> C596323; ALT1 MFR (none) -> YAGEO; ALT1 MPN (none) -> CC0805KKX7R0BB474; ALT2 LCSC (none) -> C597303; ALT2 MFR (none) -> KYOCERA AVX; ALT2 MPN (none) -> 08051C474K4Z2A; SOURCING (none) -> JLC global sourcing (first build) until an ALT is approved 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
- C17, C26: ALT NOTE (none) -> 1 µF ±10 % 100 V X7S 0805; power path: Sofar review; ALT1 LCSC (none) -> C342785; ALT1 MFR (none) -> TDK; ALT1 MPN (none) -> C2012X7S2A105KT000N; ALT2 LCSC (none) -> C126585; ALT2 MFR (none) -> Murata; ALT2 MPN (none) -> GCM21BC72A105KE36L; SOURCING (none) -> JLC global sourcing (first build) until an ALT is approved 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
- C19, C27: ALT NOTE (none) -> 1 nF 1 kV X7R 0805, ±10 % (tighter); PoDL front end: Sofar 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; ALT1 LCSC (none) -> C2167549; ALT1 MFR (none) -> KEMET; ALT1 MPN (none) -> C0805C102KDRACTU; ALT2 LCSC (none) -> C303890; ALT2 MFR (none) -> Walsin; ALT2 MPN (none) -> 0805B102K102CT; SOURCING (none) -> JLC global sourcing (first build) until an ALT is approved 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
- C21: ALT NOTE (none) -> 10 µF ±10 % 50 V X7R 1210; power path: Sofar review; ALT1 LCSC (none) -> C116808; ALT1 MFR (none) -> FH; ALT1 MPN (none) -> 1210B106K500NT; ALT2 LCSC (none) -> C386167; ALT2 MFR (none) -> Taiyo Yuden; ALT2 MPN (none) -> UMK325AB7106KM-T; SOURCING (none) -> JLC global sourcing (first build) until an ALT is approved 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
- C22, C23: ALT NOTE (none) -> Sofar review: bus damping; a newly sourced replacement must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; SOURCING (none) -> JLC global sourcing (first build) until an ALT is approved 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
- D1: SOURCING (none) -> JLC global sourcing of Sofar's second source Vishay SMA6F33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
- D2: SOURCING (none) -> JLC global sourcing (D26); no LCSC listing
- R14, R18: ALT NOTE (none) -> 100 Ω ±0.1 % ±25 ppm thin film 0402 (tighter); ALT2 AEC-Q20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; ALT1 LCSC (none) -> C705627; ALT1 MFR (none) -> YAGEO; ALT1 MPN (none) -> RT0402BRD07100RL; ALT2 LCSC (none) -> C445575; ALT2 MFR (none) -> Panasonic; ALT2 MPN (none) -> ERA2AEB101X; SOURCING (none) -> JLC global sourcing (first build) until an ALT is approved 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
- R15, R16: ALT NOTE (none) -> Sofar review: 7.5 Ω ±1 % 0.5 W, ±200 vs ±100 ppm/°C, pulse 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; ALT1 LCSC (none) -> C873769; ALT1 MFR (none) -> YAGEO; ALT1 MPN (none) -> SR0805FR-477R5L; SOURCING (none) -> JLC global sourcing (first build) until an ALT is approved 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

Commit message: S5.i: planned part per BOM line (D27) beside Sofar's specified part
- PLANNED MPN/MFR/LCSC + PLANNED NOTE (why) on all 106 purchased parts;
  Value (Sofar's part) unchanged
- 10 lines planned as LCSC-stocked equivalents (R34, R20/R39, R21 group,
  C31, C17/C26, C21, C16 group, C19/C27, R14/R18) and D1 -> Sofar's Vishay
  second source; R8 kept (no ROHM land pattern); J1 TBD; rest as specified
- SOURCING on the 19 changed-line parts: planned part after Sofar approves
- Footprint lines of U11, R41, C56-C58 re-indented (whitespace only)
- View "Sofar review (planned parts)"; check.sh exports bom.csv from it
- Fields only: ERC 531/27/504 unchanged, netcheck 51/51, midwire 0
- Docs: DESIGN D27, bom_alternates, bom_lifecycle, sofar_brief, changelog,
  TRACKER, viewer, DEV_LOG

Co-Authored-By: Claude Opus 5.5 <noreply@anthropic.com>
Parts:
- C16, C18, C24, C25: PLANNED LCSC (none) -> C596323; PLANNED MFR (none) -> YAGEO; PLANNED MPN (none) -> CC0805KKX7R0BB474; PLANNED NOTE (none) -> Same spec, 470 nF ±10 % 100 V X7R 0805, largest LCSC stock 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; SOURCING JLC global sourcing (first build) until an ALT is approved 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 -> Planned part from LCSC once Sofar approves it (D27); until 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
- C17, C26: PLANNED LCSC (none) -> C342785; PLANNED MFR (none) -> TDK; PLANNED MPN (none) -> C2012X7S2A105KT000N; PLANNED NOTE (none) -> TDK's other catalog number for the same 1 µF ±10 % 100 V X7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; SOURCING JLC global sourcing (first build) until an ALT is approved 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 -> Planned part from LCSC once Sofar approves it (D27); until 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
- C19, C27: PLANNED LCSC (none) -> C2167549; PLANNED MFR (none) -> KEMET; PLANNED MPN (none) -> C0805C102KDRACTU; PLANNED NOTE (none) -> Same KEMET series, ±10 % instead of ±20 % (tighter); 1 nF 1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; SOURCING JLC global sourcing (first build) until an ALT is approved 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 -> Planned part from LCSC once Sofar approves it (D27); until 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
- C20: PLANNED LCSC (none) -> C77058; PLANNED MFR (none) -> Murata; PLANNED MPN (none) -> GRM188R72A104KA35D; PLANNED NOTE (none) -> As specified; in LCSC stock (checked 2026-10-06)
- C21: PLANNED LCSC (none) -> C386167; PLANNED MFR (none) -> Taiyo Yuden; PLANNED MPN (none) -> UMK325AB7106KM-T; PLANNED NOTE (none) -> 10 µF ±10 % 50 V X7R 1210 from a tier-1 maker for the power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; SOURCING JLC global sourcing (first build) until an ALT is approved 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 -> Planned part from LCSC once Sofar approves it (D27); until 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
- C22, C23: PLANNED LCSC (none) -> C92059; PLANNED MFR (none) -> Panasonic; PLANNED MPN (none) -> EEEFT1H470AP; PLANNED NOTE (none) -> As specified (Sofar review): no potting-safe like-for-like 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
- D1: PLANNED MFR (none) -> Vishay; PLANNED MPN (none) -> SMA6F33A-M3/H; PLANNED NOTE (none) -> Sofar's own listed second source (their MANUFACTURERPARTNUM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
- D2: PLANNED MFR (none) -> ROHM; PLANNED MPN (none) -> RB058LAM-60TFTR; PLANNED NOTE (none) -> As specified; JLC global sourcing (D26): no LCSC listing
- D4, D5: PLANNED LCSC (none) -> C911382; PLANNED MFR (none) -> Bourns; PLANNED MPN (none) -> CDSOD323-T36SC; PLANNED NOTE (none) -> As specified; in LCSC stock (checked 2026-10-06)
- L1, L2: PLANNED LCSC (none) -> C6496096; PLANNED MFR (none) -> Bourns; PLANNED MPN (none) -> SRF1260-101M; PLANNED NOTE (none) -> As specified; in LCSC stock (checked 2026-10-06) (thin marg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
- R12, R13, R17, R19: PLANNED LCSC (none) -> C844880; PLANNED MFR (none) -> Vishay Dale; PLANNED MPN (none) -> CRCW12100000Z0EA; PLANNED NOTE (none) -> As specified; in LCSC stock (checked 2026-10-06)
- R14, R18: PLANNED LCSC (none) -> C705627; PLANNED MFR (none) -> YAGEO; PLANNED MPN (none) -> RT0402BRD07100RL; PLANNED NOTE (none) -> 100 Ω thin film 0402, ±0.1 % ±25 ppm (tighter than the spec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; SOURCING JLC global sourcing (first build) until an ALT is approved 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 -> Planned part from LCSC once Sofar approves it (D27); until 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
- R15, R16: PLANNED MFR (none) -> Vishay Dale; PLANNED MPN (none) -> CRCW08057R50FKEAHP; PLANNED NOTE (none) -> As specified (Sofar review): the only stocked alternate (YA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
- T1, T2: PLANNED LCSC (none) -> C4354923; PLANNED MFR (none) -> Würth Elektronik; PLANNED MPN (none) -> 74930000; PLANNED NOTE (none) -> As specified; in LCSC stock (checked 2026-10-06)

Commit message: S5.i: QE round 1 APPROVED WITH NITS -- notes fixed; record report; S5 complete
- F1: R21 group "ample LCSC stock"; C16 group stock figures stated
- N1: C17/C26 note no longer claims the same part (thickness not confirmed)
- N2: D26 marked "amended by D27"; N3: C21 note reworded
- R8 datasheet URLs in bom_alternates.md
- QE report in docs/design-review/qe/S5.md; TRACKER, viewer, DEV_LOG

Co-Authored-By: Claude Opus 5.5 <noreply@anthropic.com>
Parts:
- C16, C18, C24, C25: PLANNED NOTE Same spec, 470 nF ±10 % 100 V X7R 0805, largest LCSC stock (the AVX ALT2 has too few for 80); specified AVX has no LCSC listing; PoDL front end: Sofar review -> Same spec, 470 nF ±10 % 100 V X7R 0805, largest LCSC stock (250,730 vs the AVX ALT2's 750, 2026-10-06); specified AVX has no LCSC listing; PoDL front end: Sofar review
- C17, C26: PLANNED NOTE TDK's other catalog number for the same 1 µF ±10 % 100 V X7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 -> TDK C2012 series, same 1 µF ±10 % 100 V X7S 0805 per LCSC (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
- C21: PLANNED NOTE 10 µF ±10 % 50 V X7R 1210 from a tier-1 maker for the power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 -> 10 µF ±10 % 50 V X7R 1210 from Taiyo Yuden, an established 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
Changed lines of the file:
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@@
 			)
 		)
-		(property "PLANNED NOTE" "Same spec, 470 nF ±10 % 100 V X7R 0805, largest LCSC stock (the AVX ALT2 has too few for 80); specified AVX has no LCSC listing; PoDL front end: Sofar review"
+		(property "PLANNED NOTE" "Same spec, 470 nF ±10 % 100 V X7R 0805, largest LCSC stock (250,730 vs the AVX ALT2's 750, 2026-10-06); specified AVX has no LCSC listing; PoDL front end: Sofar review"
 			(at 60.96 192.8622 0)
 			(effects
@@
 			)
 		)
-		(property "PLANNED NOTE" "Same spec, 470 nF ±10 % 100 V X7R 0805, largest LCSC stock (the AVX ALT2 has too few for 80); specified AVX has no LCSC listing; PoDL front end: Sofar review"
+		(property "PLANNED NOTE" "Same spec, 470 nF ±10 % 100 V X7R 0805, largest LCSC stock (250,730 vs the AVX ALT2's 750, 2026-10-06); specified AVX has no LCSC listing; PoDL front end: Sofar review"
 			(at 116.84 116.6622 0)
 			(effects
@@
 			)
 		)
-		(property "PLANNED NOTE" "Same spec, 470 nF ±10 % 100 V X7R 0805, largest LCSC stock (the AVX ALT2 has too few for 80); specified AVX has no LCSC listing; PoDL front end: Sofar review"
+		(property "PLANNED NOTE" "Same spec, 470 nF ±10 % 100 V X7R 0805, largest LCSC stock (250,730 vs the AVX ALT2's 750, 2026-10-06); specified AVX has no LCSC listing; PoDL front end: Sofar review"
 			(at 116.84 228.4222 0)
 			(effects
@@
 			)
 		)
-		(property "PLANNED NOTE" "TDK's other catalog number for the same 1 µF ±10 % 100 V X7S 0805 (same C2012X7S2A105K base); specified number out of stock at LCSC; power path: Sofar review"
+		(property "PLANNED NOTE" "TDK C2012 series, same 1 µF ±10 % 100 V X7S 0805 per LCSC (thickness not confirmed: K125AB is 1.25 mm, KT000N doesn't state it); specified number out of stock at LCSC; power path: Sofar review"
 			(at 203.2 228.4222 0)
 			(effects
@@
 			)
 		)
-		(property "PLANNED NOTE" "10 µF ±10 % 50 V X7R 1210 from a tier-1 maker for the power path (FH ALT1 has more stock, kept as backup); specified Samsung out of stock at LCSC and DK; Sofar review"
+		(property "PLANNED NOTE" "10 µF ±10 % 50 V X7R 1210 from Taiyo Yuden, an established MLCC maker, for the power path (FH ALT1 has more stock, kept as backup); specified Samsung out of stock at LCSC and DK; Sofar review"
 			(at 299.72 142.0622 0)
 			(effects
@@
 			)
 		)
-		(property "PLANNED NOTE" "Same spec, 470 nF ±10 % 100 V X7R 0805, largest LCSC stock (the AVX ALT2 has too few for 80); specified AVX has no LCSC listing; PoDL front end: Sofar review"
+		(property "PLANNED NOTE" "Same spec, 470 nF ±10 % 100 V X7R 0805, largest LCSC stock (250,730 vs the AVX ALT2's 750, 2026-10-06); specified AVX has no LCSC listing; PoDL front end: Sofar review"
 			(at 60.96 81.1022 0)
 			(effects
@@
 			)
 		)
-		(property "PLANNED NOTE" "TDK's other catalog number for the same 1 µF ±10 % 100 V X7S 0805 (same C2012X7S2A105K base); specified number out of stock at LCSC; power path: Sofar review"
+		(property "PLANNED NOTE" "TDK C2012 series, same 1 µF ±10 % 100 V X7S 0805 per LCSC (thickness not confirmed: K125AB is 1.25 mm, KT000N doesn't state it); specified number out of stock at LCSC; power path: Sofar review"
 			(at 208.28 93.8022 0)
 			(effects
