File: nereus_Pi_shield_ADIN2111/BM_Mote_1_PoDL.kicad_sch (KiCad schematic)
At the start: 28 parts, among them T1 74930000, T2 74930000

Commit message: S6.a: BOM hygiene -- TP/FID/MTG out of the BOM; MANUFACTURER filled
- in_bom no on TP x16, FID1-6, MTG1-4 (bare copper / holes)
- MANUFACTURER on the 75 BOM parts without one, from bom_lifecycle.md;
  Sofar's MFR_NAME / MANUFACTURER1 / MANUFACTURER 1 untouched; J1 open
- bom.csv 51 rows, Mfr on every row but J1
- ERC 531/27/504 unchanged, netcheck 51/51, midwire 0
- Docs: bom_lifecycle, changelog, DESIGN, TRACKER (S6 bites), viewer, DEV_LOG

Co-Authored-By: Claude Opus 5.5 <noreply@anthropic.com>
Parts:
- C16, C18, C24, C25: MANUFACTURER (none) -> KYOCERA AVX
- C17, C26: MANUFACTURER (none) -> TDK
- C20: MANUFACTURER (none) -> Murata
- C21: MANUFACTURER (none) -> Samsung
- C22, C23: MANUFACTURER (none) -> Panasonic
- D1: MANUFACTURER (none) -> STMicroelectronics
- D2: MANUFACTURER (none) -> ROHM
- L1, L2: MANUFACTURER (none) -> Bourns
- R12, R13, R17, R19: MANUFACTURER (none) -> Vishay Dale
- R14, R18: MANUFACTURER (none) -> Susumu
- T1, T2: MANUFACTURER (none) -> Würth Elektronik
Changed lines of the file:
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@@
 			)
 		)
+		(property "MANUFACTURER" "Bourns"
+			(at 238.76 223.3422 0)
+			(effects
+				(font
+					(size 1.27 1.27)
+				)
+				(hide yes)
+			)
+		)
 		(pin "1"
 		)
@@
 			)
 		)
+		(property "MANUFACTURER" "KYOCERA AVX"
+			(at 60.96 192.8622 0)
+			(effects
+				(font
+					(size 1.27 1.27)
+				)
+				(hide yes)
+			)
+		)
 		(pin "1"
 		)
@@
 			)
 		)
+		(property "MANUFACTURER" "Vishay Dale"
+			(at 256.54 103.9622 0)
+			(effects
+				(font
+					(size 1.27 1.27)
+				)
+				(hide yes)
+			)
+		)
 		(pin "1"
 		)
@@
 			)
 		)
+		(property "MANUFACTURER" "Susumu"
+			(at 60.96 103.9622 0)
+			(effects
+				(font
+					(size 1.27 1.27)
+				)
+				(hide yes)
+			)
+		)
 		(pin "1"
 		)
@@
 			)
 		)
+		(property "MANUFACTURER" "KYOCERA AVX"
+			(at 116.84 116.6622 0)
+			(effects
+				(font
+					(size 1.27 1.27)
+				)
+				(hide yes)
+			)
+		)
 		(pin "1"
 		)
@@
 			)
 		)
+		(property "MANUFACTURER" "Würth Elektronik"
+			(at 101.6 70.9422 0)
+			(effects
+				(font
+					(size 1.27 1.27)
+				)
+				(hide yes)
+			)
+		)
 		(pin "1"
 		)
@@
 			)
 		)
+		(property "MANUFACTURER" "Panasonic"
+			(at 312.42 147.1422 0)
+			(effects
+				(font
+					(size 1.27 1.27)
+				)
+				(hide yes)
+			)
+		)
 		(pin "1"
 		)
@@
 			)
 		)
+		(property "MANUFACTURER" "KYOCERA AVX"
+			(at 116.84 228.4222 0)
+			(effects
+				(font
+					(size 1.27 1.27)
+				)
+				(hide yes)
+			)
+		)
 		(pin "1"
 		)
@@
 			)
 		)
+		(property "MANUFACTURER" "Vishay Dale"
+			(at 256.54 73.4822 0)
+			(effects
+				(font
+					(size 1.27 1.27)
+				)
+				(hide yes)
+			)
+		)
 		(pin "1"
 		)
@@
 			)
 		)
+		(property "MANUFACTURER" "Vishay Dale"
+			(at 256.54 208.1022 0)
+			(effects
+				(font
+					(size 1.27 1.27)
+				)
+				(hide yes)
+			)
+		)
 		(pin "1"
 		)
@@
 			)
 		)
+		(property "MANUFACTURER" "Murata"
+			(at 287.02 142.0622 0)
+			(effects
+				(font
+					(size 1.27 1.27)
+				)
+				(hide yes)
+			)
+		)
 		(pin "1"
 		)
@@
 			)
 		)
+		(property "MANUFACTURER" "TDK"
+			(at 203.2 228.4222 0)
+			(effects
+				(font
+					(size 1.27 1.27)
+				)
+				(hide yes)
+			)
+		)
 		(pin "1"
 		)
@@
 			)
 		)
+		(property "MANUFACTURER" "Samsung"
+			(at 299.72 142.0622 0)
+			(effects
+				(font
+					(size 1.27 1.27)
+				)
+				(hide yes)
+			)
+		)
 		(pin "1"
 		)
@@
 			)
 		)
+		(property "MANUFACTURER" "KYOCERA AVX"
+			(at 60.96 81.1022 0)
+			(effects
+				(font
+					(size 1.27 1.27)
+				)
+				(hide yes)
+			)
+		)
 		(pin "1"
 		)
@@
 			)
 		)
+		(property "MANUFACTURER" "TDK"
+			(at 208.28 93.8022 0)
+			(effects
+				(font
+					(size 1.27 1.27)
+				)
+				(hide yes)
+			)
+		)
 		(pin "2"
 		)
@@
 			)
 		)
+		(property "MANUFACTURER" "Susumu"
+			(at 60.96 215.7222 0)
+			(effects
+				(font
+					(size 1.27 1.27)
+				)
+				(hide yes)
+			)
+		)
 		(pin "1"
 		)
@@
 			)
 		)
+		(property "MANUFACTURER" "ROHM"
+			(at 383.54 152.2222 0)
+			(effects
+				(font
+					(size 1.27 1.27)
+				)
+				(hide yes)
+			)
+		)
 		(pin "2"
 		)
@@
 			)
 		)
+		(property "MANUFACTURER" "Vishay Dale"
+			(at 256.54 238.5822 0)
+			(effects
+				(font
+					(size 1.27 1.27)
+				)
+				(hide yes)
+			)
+		)
 		(pin "1"
 		)
@@
 			)
 		)
+		(property "MANUFACTURER" "Würth Elektronik"
+			(at 101.6 182.7022 0)
+			(effects
+				(font
+					(size 1.27 1.27)
+				)
+				(hide yes)
+			)
+		)
 		(pin "4"
 		)
@@
 			)
 		)
+		(property "MANUFACTURER" "Panasonic"
+			(at 335.28 147.1422 0)
+			(effects
+				(font
+					(size 1.27 1.27)
+				)
+				(hide yes)
+			)
+		)
 		(pin "1"
 		)
@@
 			)
 		)
+		(property "MANUFACTURER" "STMicroelectronics"
+			(at 358.14 144.6022 0)
+			(effects
+				(font
+					(size 1.27 1.27)
+				)
+				(hide yes)
+			)
+		)
 		(pin "1"
 		)
@@
 			(at 238.76 88.7222 0)
 			(effects
+				(font
+					(size 1.27 1.27)
+				)
+				(hide yes)
+			)
+		)
+		(property "MANUFACTURER" "Bourns"
+			(at 238.76 88.7222 0)
+			(effects
