File: nereus_Pi_shield_ADIN2111/BM_Mote_1_PoDL.kicad_sch (KiCad schematic)
At the start: 28 parts, among them T1 74930000, T2 74930000

Commit message: S6.g: presentation clean-up (Nick's list) + active-low names (D30)
- Top-Level: VBUS_OUT beside the Load Switch; I2C page-long runs ->
  labelled stubs at the PoDL pins; R43 beside the ADIN HW_EN pin; J5
  spaced with its note
- Cover: mote renders + old index -> grey TBD box + real sheet index;
  dimensions TBD; revision table inside the page, about this board;
  licence note and CC logo clear of the title block
- ADIN: supplies and LED blocks spaced from U1A, with headers
- Power: 3V3 / 1V8 / 5V converters spaced, with headers
- All sheets: KiCad title block filled; Altium overlay texts removed
- Names: ~{ADIN_RST}, ~{ADIN_INT}, ~{ADIN_CS}, ~{ADIN_P1/P2_LED1},
  PAYLOAD_EN, ~{PAYLOAD_FAULT} (labels, hier labels, sheet pins)
- Same pin partition; ERC 495 -> 492 / 0 errors; 8 exclusion keys
  regenerated (reasons unchanged); netcheck 51/51; midwire 0
- Docs: DESIGN D30 + pin map, changelog, README, sofar_brief, TRACKER,
  viewer, DEV_LOG; schematic.pdf re-exported

Co-Authored-By: Claude Opus 5.5 <noreply@anthropic.com>
Other:
- note removed: "${##}"
- note removed: "${#}"
- note removed: "${AUTHOR}"
- note removed: "${PCBPARTNUMBER}"
- note removed: "${REVISION}"
- note removed: "${TITLE}"
Changed lines of the file:
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@@
 	(title_block
 		(title "PoDL (Power over Data Line)")
+		(date "2026-10-07")
 		(rev "AA")
+		(comment 1 "${PCBPARTNAME} · ${PCBPARTNUMBER}")
+		(comment 2 "Author: ${AUTHOR}")
+		(comment 3 "Derived from Sofar Bristlemouth mote 000639-AB")
 	)
 	(text "Coupling Network - Port 2"
@@
 		)
 	)
-	(text "${REVISION}"
-		(exclude_from_sim no)
-		(at 410.21 285.5722 0)
-		(effects
-			(font
-				(size 1.27 1.27)
-			)
-			(justify left bottom)
-		)
-	)
 	(text "Snubber resistors must be at least 1/2 W, to support hot-plugging."
 		(exclude_from_sim no)
@@
 		)
 	)
-	(text "${#}"
-		(exclude_from_sim no)
-		(at 395.224 289.3822 0)
-		(effects
-			(font
-				(size 1.27 1.27)
-			)
-			(justify left bottom)
-		)
-	)
 	(text "Port 2"
 		(exclude_from_sim no)
@@
 			(font
 				(size 3.048 3.048)
-			)
-			(justify left bottom)
-		)
-	)
-	(text "${AUTHOR}"
-		(exclude_from_sim no)
-		(at 401.32 291.9222 0)
-		(effects
-			(font
-				(size 1.27 1.27)
 			)
 			(justify left bottom)
@@
 			)
 			(justify left bottom)
-		)
-	)
-	(text "${PCBPARTNUMBER}"
-		(exclude_from_sim no)
-		(at 356.87 285.5722 0)
-		(effects
-			(font
-				(size 1.27 1.27)
-			)
-			(justify left bottom)
-		)
-	)
-	(text "${TITLE}"
-		(exclude_from_sim no)
-		(at 356.108 277.4442 0)
-		(effects
-			(font
-				(size 1.778 1.778)
-			)
-			(justify left bottom)
-		)
-	)
-	(text "${##}"
-		(exclude_from_sim no)
-		(at 400.05 289.3822 0)
-		(effects
-			(font
-				(size 1.27 1.27)
-			)
-			(justify left bottom)
