File: nereus_Pi_shield_ADIN2111/BM_Mote_1_Power.kicad_sch (KiCad schematic)
At the start: 26 parts, among them U10 LMR51430YDDCR, U5 LMR51430YDDCR, U6 TPS62840YBGR

Commit message: S4.d: footprints findable -- project library Vault (mote.pretty) extracted from the mote board; close S5.a
43 footprints the schematic uses, extracted read-only from the reference
board with KiCad 9.0.6 pcbnew (tools/fpextract.py, back-side parts
flipped, nets cleared), registered as nickname Vault to match the board
IDs; 118 bare footprint fields -> Vault:<name>. fpextract --verify: 0
problems (negative-tested). Netlist identical except footprint fields.
ERC 74/626 -> 74/508 (footprint-link warnings gone). D19.

Co-Authored-By: Claude Opus 5.5 <noreply@anthropic.com>
Parts:
- C28, C53: footprint FP-CL278-IPC_C -> Vault:FP-CL278-IPC_C
- C29, C54: footprint FP-GRM188-0_1-e0_2_0_5-IPC_B -> Vault:FP-GRM188-0_1-e0_2_0_5-IPC_B
- C30, C55: footprint FP-0603-L_1_6_0_2-W_0_8_0-MFG -> Vault:FP-0603-L_1_6_0_2-W_0_8_0-MFG
- C31: footprint CAPC1608X100X20ML10 -> Vault:CAPC1608X100X20ML10
- C32: footprint FP-GRJ155-0_2-MFG -> Vault:FP-GRJ155-0_2-MFG
- C33: footprint FP-GRM155-0_15-MFG -> Vault:FP-GRM155-0_15-MFG
- L3, L6: footprint FP-PA5432_472NLT-MFG -> Vault:FP-PA5432_472NLT-MFG
- L4: footprint FP-DFE201612C-MFG -> Vault:FP-DFE201612C-MFG
- R20, R39: footprint FP-CRCW0402-e3-MFG -> Vault:FP-CRCW0402-e3-MFG
- R21, R37: footprint FP-RMCF0402-IPC_C -> Vault:FP-RMCF0402-IPC_C
- R22, R40: footprint RESC1005X40X25LL05T10 -> Vault:RESC1005X40X25LL05T10
- R23, R38: footprint FP-RC0402-0_4-IPC_B -> Vault:FP-RC0402-0_4-IPC_B
- U10, U5: footprint SOT-23-THIN-6_DDC_TEX -> Vault:SOT-23-THIN-6_DDC_TEX
- U6: footprint FP-YBG0006-MFG -> Vault:FP-YBG0006-MFG
Changed lines of the file:
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@@
 			)
 		)
-		(property "Footprint" ""
+				(property "Footprint" ""
 			(at 313.69 191.5922 0)
 			(effects
@@
 			)
 		)
-		(property "Footprint" ""
+				(property "Footprint" ""
 			(at 102.87 138.2522 0)
 			(effects
@@
 			)
 		)
-		(property "Footprint" "FP-GRJ155-0_2-MFG"
+		(property "Footprint" "Vault:FP-GRJ155-0_2-MFG"
 			(at 336.55 182.7022 0)
 			(effects
@@
 			)
 		)
-		(property "Footprint" "FP-YBG0006-MFG"
+		(property "Footprint" "Vault:FP-YBG0006-MFG"
 			(at 278.13 176.3522 0)
 			(effects
@@
 			)
 		)
-		(property "Footprint" "FP-CL278-IPC_C"
+		(property "Footprint" "Vault:FP-CL278-IPC_C"
 			(at 177.8 129.3622 0)
 			(effects
@@
 			)
 		)
-		(property "Footprint" "CAPC1608X100X20ML10"
+		(property "Footprint" "Vault:CAPC1608X100X20ML10"
 			(at 205.74 145.8722 0)
 			(effects
@@
 			)
 		)
-		(property "Footprint" ""
+				(property "Footprint" ""
 			(at 74.93 166.1922 0)
 			(effects
@@
 			)
 		)
-		(property "Footprint" ""
+				(property "Footprint" ""
 			(at 232.41 182.7022 0)
 			(effects
@@
 			)
 		)
-		(property "Footprint" "FP-DFE201612C-MFG"
+		(property "Footprint" "Vault:FP-DFE201612C-MFG"
 			(at 313.69 176.3522 0)
 			(effects
@@
 			)
 		)
-		(property "Footprint" "FP-PA5432_472NLT-MFG"
+		(property "Footprint" "Vault:FP-PA5432_472NLT-MFG"
 			(at 187.96 134.4422 0)
 			(effects
@@
 			)
 		)
-		(property "Footprint" "SOT-23-THIN-6_DDC_TEX"
+		(property "Footprint" "Vault:SOT-23-THIN-6_DDC_TEX"
 			(at 128.27 131.9022 0)
 			(effects
@@
 			)
 		)
-		(property "Footprint" "FP-CRCW0402-e3-MFG"
+		(property "Footprint" "Vault:FP-CRCW0402-e3-MFG"
 			(at 74.93 150.9522 0)
 			(effects
@@
 			)
 		)
-		(property "Footprint" "RESC1005X40X25LL05T10"
+		(property "Footprint" "Vault:RESC1005X40X25LL05T10"
 			(at 72.39 163.6522 0)
 			(effects
@@
 			)
 		)
-		(property "Footprint" "FP-GRM155-0_15-MFG"
+		(property "Footprint" "Vault:FP-GRM155-0_15-MFG"
 			(at 256.54 183.9722 0)
 			(effects
@@
 			)
 		)
-		(property "Footprint" ""
+				(property "Footprint" ""
 			(at 205.74 148.4122 0)
 			(effects
@@
 			)
 		)
-		(property "Footprint" "FP-RMCF0402-IPC_C"
+		(property "Footprint" "Vault:FP-RMCF0402-IPC_C"
 			(at 232.41 136.9822 0)
 			(effects
@@
 			)
 		)
-		(property "Footprint" ""
+				(property "Footprint" ""
 			(at 95.25 138.2522 0)
 			(effects
@@
 			)
 		)
-		(property "Footprint" "FP-RC0402-0_4-IPC_B"
+		(property "Footprint" "Vault:FP-RC0402-0_4-IPC_B"
 			(at 232.41 164.9222 0)
 			(effects
@@
 			)
 		)
-		(property "Footprint" ""
+				(property "Footprint" ""
 			(at 256.54 191.5922 0)
 			(effects
@@
 			)
 		)
-		(property "Footprint" ""
+				(property "Footprint" ""
 			(at 336.55 191.5922 0)
 			(effects
@@
 			)
 		)
-		(property "Footprint" "FP-GRM188-0_1-e0_2_0_5-IPC_B"
+		(property "Footprint" "Vault:FP-GRM188-0_1-e0_2_0_5-IPC_B"
 			(at 95.25 133.1722 0)
 			(effects
@@
 			)
 		)
-		(property "Footprint" "FP-0603-L_1_6_0_2-W_0_8_0-MFG"
+		(property "Footprint" "Vault:FP-0603-L_1_6_0_2-W_0_8_0-MFG"
 			(at 102.87 133.1722 0)
 			(effects
@@
 			)
 		)
-		(property "Footprint" ""
+				(property "Footprint" ""
 			(at 125.73 142.0622 0)
 			(effects
@@
 			)
 		)
-		(property "Footprint" ""
+				(property "Footprint" ""
 			(at 275.59 191.5922 0)
 			(effects
@@
 			)
 		)
-		(property "Footprint" ""
+				(property "Footprint" ""
 			(at 102.87 214.4522 0)
 			(effects
@@
 			)
 		)
-		(property "Footprint" "FP-CL278-IPC_C"
+		(property "Footprint" "Vault:FP-CL278-IPC_C"
 			(at 177.8 205.5622 0)
 			(effects
@@
 			)
 		)
-		(property "Footprint" "Capacitor_SMD:C_0805_2012Metric"
+				(property "Footprint" "Capacitor_SMD:C_0805_2012Metric"
 			(at 205.74 222.0722 0)
 			(effects
@@
 			)
 		)
-		(property "Footprint" ""
+				(property "Footprint" ""
 			(at 74.93 242.3922 0)
 			(effects
@@
 			)
 		)
-		(property "Footprint" ""
+				(property "Footprint" ""
 			(at 232.41 258.9022 0)
 			(effects
@@
 			)
 		)
-		(property "Footprint" "FP-PA5432_472NLT-MFG"
+		(property "Footprint" "Vault:FP-PA5432_472NLT-MFG"
 			(at 187.96 210.6422 0)
 			(effects
@@
 			)
 		)
-		(property "Footprint" "SOT-23-THIN-6_DDC_TEX"
+		(property "Footprint" "Vault:SOT-23-THIN-6_DDC_TEX"
 			(at 128.27 208.1022 0)
 			(effects
@@
 			)
 		)
-		(property "Footprint" "FP-CRCW0402-e3-MFG"
+		(property "Footprint" "Vault:FP-CRCW0402-e3-MFG"
 			(at 74.93 227.1522 0)
 			(effects
@@
 			)
 		)
-		(property "Footprint" "RESC1005X40X25LL05T10"
+		(property "Footprint" "Vault:RESC1005X40X25LL05T10"
 			(at 72.39 239.8522 0)
 			(effects
@@
 			)
 		)
-		(property "Footprint" ""
+				(property "Footprint" ""
 			(at 205.74 224.6122 0)
 			(effects
@@
 			)
 		)
-		(property "Footprint" "FP-RMCF0402-IPC_C"
+		(property "Footprint" "Vault:FP-RMCF0402-IPC_C"
 			(at 232.41 213.1822 0)
 			(effects
@@
 			)
 		)
-		(property "Footprint" ""
+				(property "Footprint" ""
 			(at 95.25 214.4522 0)
 			(effects
@@
 			)
 		)
-		(property "Footprint" "FP-RC0402-0_4-IPC_B"
+		(property "Footprint" "Vault:FP-RC0402-0_4-IPC_B"
 			(at 232.41 241.1222 0)
 			(effects
@@
 			)
 		)
-		(property "Footprint" "FP-GRM188-0_1-e0_2_0_5-IPC_B"
+		(property "Footprint" "Vault:FP-GRM188-0_1-e0_2_0_5-IPC_B"
 			(at 95.25 209.3722 0)
 			(effects
@@
 			)
 		)
-		(property "Footprint" "FP-0603-L_1_6_0_2-W_0_8_0-MFG"
+		(property "Footprint" "Vault:FP-0603-L_1_6_0_2-W_0_8_0-MFG"
 			(at 102.87 209.3722 0)
 			(effects
@@
 			)
 		)
-		(property "Footprint" ""
+				(property "Footprint" ""
 			(at 125.73 218.2622 0)
 			(effects
@@
 			)
 		)
-		(property "Footprint" "Capacitor_SMD:C_0805_2012Metric"
+				(property "Footprint" "Capacitor_SMD:C_0805_2012Metric"
 			(at 241.3 222.0722 0)
 			(effects
@@
 			)
 		)
-		(property "Footprint" ""
+				(property "Footprint" ""
 			(at 241.3 224.6122 0)
 			(effects
@@
 			)
 		)
-		(property "Footprint" "Capacitor_SMD:C_0402_1005Metric"
+				(property "Footprint" "Capacitor_SMD:C_0402_1005Metric"
 			(at 254 218.2622 0)
 			(effects
@@
 			)
 		)
-		(property "Footprint" ""
+				(property "Footprint" ""
 			(at 254 225.8822 0)
 			(effects

Commit message: S5.h: BOM alternates as hidden ALT/SOURCING fields; tracked bom.csv
- 24 flagged passives: hidden ALT1/ALT2 MPN/MFR/LCSC, ALT NOTE, SOURCING
  (values from docs/design-review/bom_alternates.md, D26)
- Critical parts (U1-U3, L3/L6, Y1, D1-D3, MP1-MP4, J5, J1): SOURCING only
- tools/check.sh exports docs/design-review/bom.csv: specified part first,
  alternates beside it; grouped by Value + DNP (R11 apart from R12/R13/R17/R19)
- J1 Footprint property re-indented (whitespace; import leftover)
- Fields only: ERC 531/27/504 unchanged, netcheck 51/51, midwire 0;
  netlist diff = the 208 new fields
- Docs: bom_alternates, bom_lifecycle, sofar_brief, changelog, DESIGN,
  TRACKER, viewer, DEV_LOG

Co-Authored-By: Claude Opus 5.5 <noreply@anthropic.com>
Parts:
- C31: ALT NOTE (none) -> 22 µF ±20 % 6.3 V X5R 0603; ALT1 LCSC (none) -> C59461; ALT1 MFR (none) -> Samsung; ALT1 MPN (none) -> CL10A226MQ8NRNC; ALT2 LCSC (none) -> C77042; ALT2 MFR (none) -> Murata; ALT2 MPN (none) -> GRM188R60J226MEA0D; SOURCING (none) -> JLC global sourcing (first build) until an ALT is approved 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
- L3, L6: SOURCING (none) -> JLC global sourcing (D26); no LCSC listing
- R20, R39: ALT NOTE (none) -> 1.82 MΩ ±1 % 62.5 mW 50 V ±100 ppm; ALT1 LCSC (none) -> C166520; ALT1 MFR (none) -> RALEC; ALT1 MPN (none) -> RTT021824FTH; SOURCING (none) -> JLC global sourcing (first build) until an ALT is approved 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
- R21, R37: ALT NOTE (none) -> 100 kΩ ±1 % 62.5 mW 50 V ±100 ppm; ALT1 is JLC Basic; AEC-Q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; ALT1 LCSC (none) -> C25741; ALT1 MFR (none) -> UNI-ROYAL; ALT1 MPN (none) -> 0402WGF1003TCE; ALT2 LCSC (none) -> C60491; ALT2 MFR (none) -> YAGEO; ALT2 MPN (none) -> RC0402FR-07100KL; SOURCING (none) -> JLC global sourcing (first build) until an ALT is approved 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

Commit message: S5.i: planned part per BOM line (D27) beside Sofar's specified part
- PLANNED MPN/MFR/LCSC + PLANNED NOTE (why) on all 106 purchased parts;
  Value (Sofar's part) unchanged
- 10 lines planned as LCSC-stocked equivalents (R34, R20/R39, R21 group,
  C31, C17/C26, C21, C16 group, C19/C27, R14/R18) and D1 -> Sofar's Vishay
  second source; R8 kept (no ROHM land pattern); J1 TBD; rest as specified
- SOURCING on the 19 changed-line parts: planned part after Sofar approves
- Footprint lines of U11, R41, C56-C58 re-indented (whitespace only)
- View "Sofar review (planned parts)"; check.sh exports bom.csv from it
- Fields only: ERC 531/27/504 unchanged, netcheck 51/51, midwire 0
- Docs: DESIGN D27, bom_alternates, bom_lifecycle, sofar_brief, changelog,
  TRACKER, viewer, DEV_LOG

Co-Authored-By: Claude Opus 5.5 <noreply@anthropic.com>
Parts:
- C28, C53: PLANNED LCSC (none) -> C100072; PLANNED MFR (none) -> Samsung; PLANNED MPN (none) -> CL05A104KA5NNNC; PLANNED NOTE (none) -> As specified; in LCSC stock (checked 2026-10-06)
- C29, C54: PLANNED LCSC (none) -> C77058; PLANNED MFR (none) -> Murata; PLANNED MPN (none) -> GRM188R72A104KA35D; PLANNED NOTE (none) -> As specified; in LCSC stock (checked 2026-10-06)
- C30, C55: PLANNED LCSC (none) -> C268016; PLANNED MFR (none) -> Taiyo Yuden; PLANNED MPN (none) -> UMK107BBJ225KA-T; PLANNED NOTE (none) -> As specified; in LCSC stock (checked 2026-10-06); Taiyo Yud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
- C31: PLANNED LCSC (none) -> C59461; PLANNED MFR (none) -> Samsung; PLANNED MPN (none) -> CL10A226MQ8NRNC; PLANNED NOTE (none) -> Same spec, 22 µF ±20 % 6.3 V X5R 0603; specified TDK out of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; SOURCING JLC global sourcing (first build) until an ALT is approved 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 -> Planned part from LCSC once Sofar approves it (D27); until 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
- C32: PLANNED LCSC (none) -> C469527; PLANNED MFR (none) -> Murata; PLANNED MPN (none) -> GRJ155R60J106ME11D; PLANNED NOTE (none) -> As specified; in LCSC stock (checked 2026-10-06)
- C33: PLANNED LCSC (none) -> C76996; PLANNED MFR (none) -> Murata; PLANNED MPN (none) -> GRM155R60J475ME87D; PLANNED NOTE (none) -> As specified; in LCSC stock (checked 2026-10-06)
- C56, C57: PLANNED LCSC (none) -> C86817; PLANNED MFR (none) -> Murata; PLANNED MPN (none) -> GRM21BR61C226ME44L; PLANNED NOTE (none) -> As specified; in LCSC stock (checked 2026-10-06)
- C58: PLANNED LCSC (none) -> C335105; PLANNED MFR (none) -> Murata; PLANNED MPN (none) -> GRM155R61A475MEAAD; PLANNED NOTE (none) -> As specified; in LCSC stock (checked 2026-10-06)
- L3, L6: PLANNED MFR (none) -> Pulse (YAGEO group); PLANNED MPN (none) -> PA5432.822NLT; PLANNED NOTE (none) -> As specified; JLC global sourcing (D26): no LCSC listing
- L4: PLANNED LCSC (none) -> C337893; PLANNED MFR (none) -> Murata; PLANNED MPN (none) -> DFE201612E-2R2M=P2; PLANNED NOTE (none) -> As specified; in LCSC stock (checked 2026-10-06)
- R20, R39: PLANNED LCSC (none) -> C166520; PLANNED MFR (none) -> RALEC; PLANNED MPN (none) -> RTT021824FTH; PLANNED NOTE (none) -> Only stocked LCSC match: 1.82 MΩ ±1 % 62.5 mW 50 V ±100 ppm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; SOURCING JLC global sourcing (first build) until an ALT is approved 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 -> Planned part from LCSC once Sofar approves it (D27); until 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
- R21, R37: PLANNED LCSC (none) -> C25741; PLANNED MFR (none) -> UNI-ROYAL; PLANNED MPN (none) -> 0402WGF1003TCE; PLANNED NOTE (none) -> JLC Basic part (no extended-part fee), largest LCSC stock; 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; SOURCING JLC global sourcing (first build) until an ALT is approved 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 -> Planned part from LCSC once Sofar approves it (D27); until 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
- R22, R40: PLANNED LCSC (none) -> C114763; PLANNED MFR (none) -> Yageo; PLANNED MPN (none) -> RC0402FR-07200KL; PLANNED NOTE (none) -> As specified; in LCSC stock (checked 2026-10-06)
- R23: PLANNED LCSC (none) -> C163478; PLANNED MFR (none) -> Yageo; PLANNED MPN (none) -> RC0402FR-0722K1L; PLANNED NOTE (none) -> As specified; in LCSC stock (checked 2026-10-06)
- R38: PLANNED LCSC (none) -> C274888; PLANNED MFR (none) -> Yageo; PLANNED MPN (none) -> RC0402FR-0713K7L; PLANNED NOTE (none) -> As specified; in LCSC stock (checked 2026-10-06)
- U10, U5: PLANNED LCSC (none) -> C5210749; PLANNED MFR (none) -> Texas Instruments; PLANNED MPN (none) -> LMR51430YDDCR; PLANNED NOTE (none) -> As specified; in LCSC stock (checked 2026-10-06)
- U6: PLANNED LCSC (none) -> C2071139; PLANNED MFR (none) -> Texas Instruments; PLANNED MPN (none) -> TPS62840YBGR; PLANNED NOTE (none) -> As specified; in LCSC stock (checked 2026-10-06)

Commit message: S5.i: QE round 1 APPROVED WITH NITS -- notes fixed; record report; S5 complete
- F1: R21 group "ample LCSC stock"; C16 group stock figures stated
- N1: C17/C26 note no longer claims the same part (thickness not confirmed)
- N2: D26 marked "amended by D27"; N3: C21 note reworded
- R8 datasheet URLs in bom_alternates.md
- QE report in docs/design-review/qe/S5.md; TRACKER, viewer, DEV_LOG

Co-Authored-By: Claude Opus 5.5 <noreply@anthropic.com>
Parts:
- R21, R37: PLANNED NOTE JLC Basic part (no extended-part fee), largest LCSC stock; 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 -> JLC Basic part (no extended-part fee), ample LCSC stock; 10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
Changed lines of the file:
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@@
 			)
 		)
-		(property "PLANNED NOTE" "JLC Basic part (no extended-part fee), largest LCSC stock; 100 kΩ ±1 % 62.5 mW 50 V ±100 ppm 0402; specified Stackpole is out of stock at LCSC and is AEC-Q200, this one doesn't state it"
+		(property "PLANNED NOTE" "JLC Basic part (no extended-part fee), ample LCSC stock; 100 kΩ ±1 % 62.5 mW 50 V ±100 ppm 0402; specified Stackpole is out of stock at LCSC and is AEC-Q200, this one doesn't state it"
 			(at 232.41 136.9822 0)
 			(effects
@@
 			)
 		)
-		(property "PLANNED NOTE" "JLC Basic part (no extended-part fee), largest LCSC stock; 100 kΩ ±1 % 62.5 mW 50 V ±100 ppm 0402; specified Stackpole is out of stock at LCSC and is AEC-Q200, this one doesn't state it"
+		(property "PLANNED NOTE" "JLC Basic part (no extended-part fee), ample LCSC stock; 100 kΩ ±1 % 62.5 mW 50 V ±100 ppm 0402; specified Stackpole is out of stock at LCSC and is AEC-Q200, this one doesn't state it"
 			(at 232.41 213.1822 0)
 			(effects

Commit message: S6.a: BOM hygiene -- TP/FID/MTG out of the BOM; MANUFACTURER filled
- in_bom no on TP x16, FID1-6, MTG1-4 (bare copper / holes)
- MANUFACTURER on the 75 BOM parts without one, from bom_lifecycle.md;
  Sofar's MFR_NAME / MANUFACTURER1 / MANUFACTURER 1 untouched; J1 open
- bom.csv 51 rows, Mfr on every row but J1
- ERC 531/27/504 unchanged, netcheck 51/51, midwire 0
- Docs: bom_lifecycle, changelog, DESIGN, TRACKER (S6 bites), viewer, DEV_LOG

Co-Authored-By: Claude Opus 5.5 <noreply@anthropic.com>
Parts:
- C28, C53: MANUFACTURER (none) -> Samsung
- C29, C32, C33, C54, L4: MANUFACTURER (none) -> Murata
- C30, C55: MANUFACTURER (none) -> Taiyo Yuden
- L3, L6: MANUFACTURER (none) -> Pulse (YAGEO group)
- R20, R39: MANUFACTURER (none) -> Vishay Dale
- R21, R37: MANUFACTURER (none) -> Stackpole
- R23, R38: MANUFACTURER (none) -> Yageo
- U10, U5, U6: MANUFACTURER (none) -> Texas Instruments
Changed lines of the file:
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@@
 			)
 		)
+		(property "MANUFACTURER" "Murata"
+			(at 336.55 182.7022 0)
+			(effects
+				(font
+					(size 1.27 1.27)
+				)
+				(hide yes)
+			)
+		)
 		(pin "1"
 		)
@@
 			)
 		)
+		(property "MANUFACTURER" "Texas Instruments"
+			(at 278.13 176.3522 0)
+			(effects
+				(font
+					(size 1.27 1.27)
+				)
+				(hide yes)
+			)
+		)
 		(pin "B1"
 		)
@@
 			)
 		)
+		(property "MANUFACTURER" "Samsung"
+			(at 177.8 129.3622 0)
+			(effects
+				(font
+					(size 1.27 1.27)
+				)
+				(hide yes)
+			)
+		)
 		(pin "1"
 		)
@@
 			)
 		)
+		(property "MANUFACTURER" "Murata"
+			(at 313.69 176.3522 0)
+			(effects
+				(font
+					(size 1.27 1.27)
+				)
+				(hide yes)
+			)
+		)
 		(pin "1"
 		)
@@
 			)
 		)
+		(property "MANUFACTURER" "Pulse (YAGEO group)"
+			(at 187.96 134.4422 0)
+			(effects
+				(font
+					(size 1.27 1.27)
+				)
+				(hide yes)
+			)
+		)
 		(pin "1"
 		)
@@
 			)
 		)
+		(property "MANUFACTURER" "Texas Instruments"
+			(at 128.27 131.9022 0)
+			(effects
+				(font
+					(size 1.27 1.27)
+				)
+				(hide yes)
+			)
+		)
 		(pin "6"
 		)
@@
 			)
 		)
+		(property "MANUFACTURER" "Vishay Dale"
+			(at 74.93 150.9522 0)
+			(effects
+				(font
+					(size 1.27 1.27)
+				)
+				(hide yes)
+			)
+		)
 		(pin "1"
 		)
@@
 			)
 		)
+		(property "MANUFACTURER" "Murata"
+			(at 256.54 183.9722 0)
+			(effects
+				(font
+					(size 1.27 1.27)
+				)
+				(hide yes)
+			)
+		)
 		(pin "1"
 		)
@@
 			)
 		)
+		(property "MANUFACTURER" "Stackpole"
+			(at 232.41 136.9822 0)
+			(effects
+				(font
+					(size 1.27 1.27)
+				)
+				(hide yes)
+			)
+		)
 		(pin "2"
 		)
@@
 			)
 		)
+		(property "MANUFACTURER" "Yageo"
+			(at 232.41 164.9222 0)
+			(effects
+				(font
+					(size 1.27 1.27)
+				)
+				(hide yes)
+			)
+		)
 		(pin "1"
 		)
@@
 			)
 		)
+		(property "MANUFACTURER" "Murata"
+			(at 95.25 133.1722 0)
+			(effects
+				(font
+					(size 1.27 1.27)
+				)
+				(hide yes)
+			)
+		)
 		(pin "2"
 		)
@@
 			)
 		)
+		(property "MANUFACTURER" "Taiyo Yuden"
+			(at 102.87 133.1722 0)
+			(effects
+				(font
+					(size 1.27 1.27)
+				)
+				(hide yes)
+			)
+		)
 		(pin "1"
 		)
@@
 			)
 		)
+		(property "MANUFACTURER" "Samsung"
+			(at 177.8 205.5622 0)
+			(effects
+				(font
+					(size 1.27 1.27)
+				)
+				(hide yes)
+			)
+		)
 		(pin "1"
 		)
@@
 			)
 		)
+		(property "MANUFACTURER" "Pulse (YAGEO group)"
+			(at 187.96 210.6422 0)
+			(effects
+				(font
+					(size 1.27 1.27)
+				)
+				(hide yes)
+			)
+		)
 		(pin "1"
 		)
@@
 			)
 		)
+		(property "MANUFACTURER" "Texas Instruments"
+			(at 128.27 208.1022 0)
+			(effects
+				(font
+					(size 1.27 1.27)
+				)
+				(hide yes)
+			)
+		)
 		(pin "6"
 		)
@@
 			)
 		)
+		(property "MANUFACTURER" "Vishay Dale"
+			(at 74.93 227.1522 0)
+			(effects
+				(font
+					(size 1.27 1.27)
+				)
+				(hide yes)
+			)
+		)
 		(pin "1"
 		)
@@
 			)
 		)
+		(property "MANUFACTURER" "Stackpole"
+			(at 232.41 213.1822 0)
+			(effects
+				(font
+					(size 1.27 1.27)
+				)
+				(hide yes)
+			)
+		)
 		(pin "2"
 		)
@@
 			)
 		)
+		(property "MANUFACTURER" "Yageo"
+			(at 232.41 241.1222 0)
+			(effects
+				(font
+					(size 1.27 1.27)
+				)
+				(hide yes)
+			)
+		)
 		(pin "1"
 		)
@@
 			)
 		)
+		(property "MANUFACTURER" "Murata"
+			(at 95.25 209.3722 0)
+			(effects
+				(font
+					(size 1.27 1.27)
+				)
+				(hide yes)
+			)
+		)
 		(pin "2"
 		)
@@
 			(at 102.87 209.3722 0)
 			(effects
+				(font
+					(size 1.27 1.27)
+				)
+				(hide yes)
+			)
+		)
+		(property "MANUFACTURER" "Taiyo Yuden"
+			(at 102.87 209.3722 0)
+			(effects
