File: nereus_Pi_shield_ADIN2111/BM_Mote_1_PowerMon.kicad_sch (KiCad schematic)
At the start: 4 parts, among them U4 INA232AIDDFR

Commit message: S4.d: footprints findable -- project library Vault (mote.pretty) extracted from the mote board; close S5.a
43 footprints the schematic uses, extracted read-only from the reference
board with KiCad 9.0.6 pcbnew (tools/fpextract.py, back-side parts
flipped, nets cleared), registered as nickname Vault to match the board
IDs; 118 bare footprint fields -> Vault:<name>. fpextract --verify: 0
problems (negative-tested). Netlist identical except footprint fields.
ERC 74/626 -> 74/508 (footprint-link warnings gone). D19.

Co-Authored-By: Claude Opus 5.5 <noreply@anthropic.com>
Parts:
- C15: footprint FP-CL278-IPC_C -> Vault:FP-CL278-IPC_C
- R7: footprint FP-RC0402-0_4-IPC_C -> Vault:FP-RC0402-0_4-IPC_C
- R8: footprint RESC1608X60X55ML20T10 -> Vault:RESC1608X60X55ML20T10
- U4: footprint INA232AIDDFR-Footprint-1 -> Vault:INA232AIDDFR-Footprint-1
Changed lines of the file:
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@@
 			)
 		)
-		(property "Footprint" "INA232AIDDFR-Footprint-1"
+		(property "Footprint" "Vault:INA232AIDDFR-Footprint-1"
 			(at 208.28 152.2222 0)
 			(effects
@@
 			)
 		)
-		(property "Footprint" "FP-CL278-IPC_C"
+		(property "Footprint" "Vault:FP-CL278-IPC_C"
 			(at 187.96 164.9222 0)
 			(effects
@@
 			)
 		)
-		(property "Footprint" "FP-RC0402-0_4-IPC_C"
+		(property "Footprint" "Vault:FP-RC0402-0_4-IPC_C"
 			(at 241.3 139.5222 0)
 			(effects
@@
 			)
 		)
-		(property "Footprint" "RESC1608X60X55ML20T10"
+		(property "Footprint" "Vault:RESC1608X60X55ML20T10"
 			(at 175.26 157.3022 0)
 			(effects
@@
 			)
 		)
-		(property "Footprint" ""
+				(property "Footprint" ""
 			(at 177.8 162.3822 0)
 			(effects

Commit message: S5.h: BOM alternates as hidden ALT/SOURCING fields; tracked bom.csv
- 24 flagged passives: hidden ALT1/ALT2 MPN/MFR/LCSC, ALT NOTE, SOURCING
  (values from docs/design-review/bom_alternates.md, D26)
- Critical parts (U1-U3, L3/L6, Y1, D1-D3, MP1-MP4, J5, J1): SOURCING only
- tools/check.sh exports docs/design-review/bom.csv: specified part first,
  alternates beside it; grouped by Value + DNP (R11 apart from R12/R13/R17/R19)
- J1 Footprint property re-indented (whitespace; import leftover)
- Fields only: ERC 531/27/504 unchanged, netcheck 51/51, midwire 0;
  netlist diff = the 208 new fields
- Docs: bom_alternates, bom_lifecycle, sofar_brief, changelog, DESIGN,
  TRACKER, viewer, DEV_LOG

Co-Authored-By: Claude Opus 5.5 <noreply@anthropic.com>
Parts:
- R8: ALT NOTE (none) -> Sofar review: power-path current sense. Sofar's own 7 liste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; ALT1 LCSC (none) -> C308571; ALT1 MFR (none) -> ROHM; ALT1 MPN (none) -> PMR03EZPFU10L0; ALT2 LCSC (none) -> C5334451; ALT2 MFR (none) -> Vishay; ALT2 MPN (none) -> WSLP0603R0100FEA; SOURCING (none) -> JLC global sourcing (first build) until an ALT is approved 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
Changed lines of the file:
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@@
+			)
+		)
+		(property "ALT1 MPN" "PMR03EZPFU10L0"
+			(at 175.26 157.3022 0)
+			(effects
+				(font
+					(size 1.27 1.27)
+				)
+				(hide yes)
+			)
+		)
+		(property "ALT1 MFR" "ROHM"
+			(at 175.26 157.3022 0)
+			(effects
+				(font
+					(size 1.27 1.27)
+				)
+				(hide yes)
+			)
+		)
+		(property "ALT1 LCSC" "C308571"
+			(at 175.26 157.3022 0)
+			(effects
+				(font
+					(size 1.27 1.27)
+				)
+				(hide yes)
+			)
+		)
+		(property "ALT2 MPN" "WSLP0603R0100FEA"
+			(at 175.26 157.3022 0)
+			(effects
+				(font
+					(size 1.27 1.27)
+				)
+				(hide yes)
+			)
+		)
+		(property "ALT2 MFR" "Vishay"
+			(at 175.26 157.3022 0)
+			(effects
+				(font
+					(size 1.27 1.27)
+				)
+				(hide yes)
+			)
+		)
+		(property "ALT2 LCSC" "C5334451"
+			(at 175.26 157.3022 0)
+			(effects
+				(font
+					(size 1.27 1.27)
+				)
+				(hide yes)
+			)
+		)
+		(property "ALT NOTE" "Sofar review: power-path current sense. Sofar's own 7 listed alternates (fields MANUFACTURERPARTNUMBER1-7) not found at LCSC; check land pattern"
+			(at 175.26 157.3022 0)
+			(effects
+				(font
+					(size 1.27 1.27)
+				)
+				(hide yes)
+			)
+		)
+		(property "SOURCING" "JLC global sourcing (first build) until an ALT is approved (D26)"
+			(at 175.26 157.3022 0)
+			(effects
+				(font
+					(size 1.27 1.27)
+				)
+				(hide yes)
 			)
 		)

Commit message: S5.h: QE round 1 APPROVED WITH NITS -- nits fixed; alternates capped at 3
- R8 ALT NOTE shortened (Nick: at most 3 alternates per part; R8's 7 Sofar
  fields stay untouched, outside bom.csv)
- J1 SOURCING back to the plan's "2x20" with the multiplication sign (N1);
  C22/C23 DK-figure drop declared in the changelog (N1)
- S6 item: TP/FID/MTG rows in bom.csv for a JLC order (N2)
- QE report recorded in docs/design-review/qe/S5.md; TRACKER, viewer, DEV_LOG

Co-Authored-By: Claude Opus 5.5 <noreply@anthropic.com>
Parts:
- R8: ALT NOTE Sofar review: power-path current sense. Sofar's own 7 liste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 -> Sofar review: power-path current sense; check land pattern
Changed lines of the file:
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@@
 			)
 		)
-		(property "ALT NOTE" "Sofar review: power-path current sense. Sofar's own 7 listed alternates (fields MANUFACTURERPARTNUMBER1-7) not found at LCSC; check land pattern"
+		(property "ALT NOTE" "Sofar review: power-path current sense; check land pattern"
 			(at 175.26 157.3022 0)
 			(effects

Commit message: S5.i: planned part per BOM line (D27) beside Sofar's specified part
- PLANNED MPN/MFR/LCSC + PLANNED NOTE (why) on all 106 purchased parts;
  Value (Sofar's part) unchanged
- 10 lines planned as LCSC-stocked equivalents (R34, R20/R39, R21 group,
  C31, C17/C26, C21, C16 group, C19/C27, R14/R18) and D1 -> Sofar's Vishay
  second source; R8 kept (no ROHM land pattern); J1 TBD; rest as specified
- SOURCING on the 19 changed-line parts: planned part after Sofar approves
- Footprint lines of U11, R41, C56-C58 re-indented (whitespace only)
- View "Sofar review (planned parts)"; check.sh exports bom.csv from it
- Fields only: ERC 531/27/504 unchanged, netcheck 51/51, midwire 0
- Docs: DESIGN D27, bom_alternates, bom_lifecycle, sofar_brief, changelog,
  TRACKER, viewer, DEV_LOG

Co-Authored-By: Claude Opus 5.5 <noreply@anthropic.com>
Parts:
- C15: PLANNED LCSC (none) -> C100072; PLANNED MFR (none) -> Samsung; PLANNED MPN (none) -> CL05A104KA5NNNC; PLANNED NOTE (none) -> As specified; in LCSC stock (checked 2026-10-06)
- R7: PLANNED LCSC (none) -> C60489; PLANNED MFR (none) -> Yageo; PLANNED MPN (none) -> RC0402JR-0710KL; PLANNED NOTE (none) -> As specified; in LCSC stock (checked 2026-10-06)
- R8: PLANNED MFR (none) -> KOA Speer; PLANNED MPN (none) -> UR73D1JTTD10L0F; PLANNED NOTE (none) -> As specified (Sofar review), JLC global sourcing: no LCSC l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
- U4: PLANNED LCSC (none) -> C5447660; PLANNED MFR (none) -> Texas Instruments; PLANNED MPN (none) -> INA232AIDDFR; PLANNED NOTE (none) -> As specified; in LCSC stock (checked 2026-10-06)
Changed lines of the file:
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@@
+			)
+		)
+		(property "PLANNED MPN" "INA232AIDDFR"
+			(at 208.28 152.2222 0)
+			(effects
+				(font
+					(size 1.27 1.27)
+				)
+				(hide yes)
+			)
+		)
+		(property "PLANNED MFR" "Texas Instruments"
+			(at 208.28 152.2222 0)
+			(effects
+				(font
+					(size 1.27 1.27)
+				)
+				(hide yes)
+			)
+		)
+		(property "PLANNED LCSC" "C5447660"
+			(at 208.28 152.2222 0)
+			(effects
+				(font
+					(size 1.27 1.27)
+				)
+				(hide yes)
+			)
+		)
+		(property "PLANNED NOTE" "As specified; in LCSC stock (checked 2026-10-06)"
+			(at 208.28 152.2222 0)
+			(effects
+				(font
+					(size 1.27 1.27)
+				)
+				(hide yes)
 			)
 		)
@@
 			)
 		)
+		(property "PLANNED MPN" "CL05A104KA5NNNC"
+			(at 187.96 164.9222 0)
+			(effects
+				(font
+					(size 1.27 1.27)
+				)
+				(hide yes)
+			)
+		)
+		(property "PLANNED MFR" "Samsung"
+			(at 187.96 164.9222 0)
+			(effects
+				(font
+					(size 1.27 1.27)
+				)
+				(hide yes)
+			)
+		)
+		(property "PLANNED LCSC" "C100072"
+			(at 187.96 164.9222 0)
+			(effects
+				(font
+					(size 1.27 1.27)
+				)
+				(hide yes)
+			)
+		)
+		(property "PLANNED NOTE" "As specified; in LCSC stock (checked 2026-10-06)"
+			(at 187.96 164.9222 0)
+			(effects
+				(font
+					(size 1.27 1.27)
+				)
+				(hide yes)
+			)
+		)
 		(pin "1"
 		)
@@
 			)
 		)
+		(property "PLANNED MPN" "RC0402JR-0710KL"
+			(at 241.3 139.5222 0)
+			(effects
+				(font
+					(size 1.27 1.27)
+				)
+				(hide yes)
+			)
+		)
+		(property "PLANNED MFR" "Yageo"
+			(at 241.3 139.5222 0)
+			(effects
+				(font
+					(size 1.27 1.27)
+				)
+				(hide yes)
+			)
+		)
+		(property "PLANNED LCSC" "C60489"
+			(at 241.3 139.5222 0)
+			(effects
+				(font
+					(size 1.27 1.27)
+				)
+				(hide yes)
+			)
+		)
+		(property "PLANNED NOTE" "As specified; in LCSC stock (checked 2026-10-06)"
+			(at 241.3 139.5222 0)
+			(effects
+				(font
+					(size 1.27 1.27)
+				)
+				(hide yes)
+			)
+		)
 		(pin "1"
 		)
@@
 			(at 175.26 157.3022 0)
 			(effects
+				(font
+					(size 1.27 1.27)
+				)
+				(hide yes)
+			)
+		)
+		(property "PLANNED MPN" "UR73D1JTTD10L0F"
+			(at 175.26 157.3022 0)
+			(effects
+				(font
+					(size 1.27 1.27)
+				)
+				(hide yes)
+			)
+		)
+		(property "PLANNED MFR" "KOA Speer"
+			(at 175.26 157.3022 0)
+			(effects
+				(font
+					(size 1.27 1.27)
+				)
+				(hide yes)
+			)
+		)
+		(property "PLANNED LCSC" ""
+			(at 175.26 157.3022 0)
+			(effects
+				(font
+					(size 1.27 1.27)
+				)
+				(hide yes)
+			)
+		)
+		(property "PLANNED NOTE" "As specified (Sofar review), JLC global sourcing: no LCSC listing. ROHM PMR03 (ALT1) electrodes (b 0.35 mm, datasheet Rev.PMR03-IA-012E) sit inside these pads, which were drawn for the UR73D1J's 0.55 mm electrodes and reach 0.35 mm under the PMR03 body; ROHM gives no land pattern, so not adopted"
+			(at 175.26 157.3022 0)
+			(effects

Commit message: S6.a: BOM hygiene -- TP/FID/MTG out of the BOM; MANUFACTURER filled
- in_bom no on TP x16, FID1-6, MTG1-4 (bare copper / holes)
- MANUFACTURER on the 75 BOM parts without one, from bom_lifecycle.md;
  Sofar's MFR_NAME / MANUFACTURER1 / MANUFACTURER 1 untouched; J1 open
- bom.csv 51 rows, Mfr on every row but J1
- ERC 531/27/504 unchanged, netcheck 51/51, midwire 0
- Docs: bom_lifecycle, changelog, DESIGN, TRACKER (S6 bites), viewer, DEV_LOG

Co-Authored-By: Claude Opus 5.5 <noreply@anthropic.com>
Parts:
- C15: MANUFACTURER (none) -> Samsung
- R7: MANUFACTURER (none) -> Yageo
- U4: MANUFACTURER (none) -> Texas Instruments
Changed lines of the file:
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@@
+			)
+		)
+		(property "MANUFACTURER" "Texas Instruments"
+			(at 208.28 152.2222 0)
+			(effects
+				(font
+					(size 1.27 1.27)
+				)
+				(hide yes)
 			)
 		)
@@
 			)
 		)
+		(property "MANUFACTURER" "Samsung"
+			(at 187.96 164.9222 0)
+			(effects
+				(font
+					(size 1.27 1.27)
+				)
+				(hide yes)
+			)
+		)
 		(pin "1"
 		)
@@
 			(at 241.3 139.5222 0)
 			(effects
+				(font
+					(size 1.27 1.27)
+				)
+				(hide yes)
+			)
+		)
+		(property "MANUFACTURER" "Yageo"
+			(at 241.3 139.5222 0)
+			(effects
