File: nereus_Pi_shield_ADIN2111/BM_Mote_1_ADIN2111.kicad_sch (KiCad schematic)
At the start: 33 parts, among them U1 ADIN2111BCPZ, U2 AP22913CN4-7, U3 AP22913CN4-7, Y1 ABM11W-25.0000MHZ-6-K1Z-T3

Commit message: S6.g: presentation clean-up (Nick's list) + active-low names (D30)
- Top-Level: VBUS_OUT beside the Load Switch; I2C page-long runs ->
  labelled stubs at the PoDL pins; R43 beside the ADIN HW_EN pin; J5
  spaced with its note
- Cover: mote renders + old index -> grey TBD box + real sheet index;
  dimensions TBD; revision table inside the page, about this board;
  licence note and CC logo clear of the title block
- ADIN: supplies and LED blocks spaced from U1A, with headers
- Power: 3V3 / 1V8 / 5V converters spaced, with headers
- All sheets: KiCad title block filled; Altium overlay texts removed
- Names: ~{ADIN_RST}, ~{ADIN_INT}, ~{ADIN_CS}, ~{ADIN_P1/P2_LED1},
  PAYLOAD_EN, ~{PAYLOAD_FAULT} (labels, hier labels, sheet pins)
- Same pin partition; ERC 495 -> 492 / 0 errors; 8 exclusion keys
  regenerated (reasons unchanged); netcheck 51/51; midwire 0
- Docs: DESIGN D30 + pin map, changelog, README, sofar_brief, TRACKER,
  viewer, DEV_LOG; schematic.pdf re-exported

Co-Authored-By: Claude Opus 5.5 <noreply@anthropic.com>
Connections:
- net ADIN_P1_LED1 renamed ~{ADIN_P1_LED1}
- net ADIN_P2_LED1 renamed ~{ADIN_P2_LED1}
Other:
- note added: "ADIN2111 status LEDs: power, port 1 / port 2 link-activity"
- note added: "ADIN2111 supplies: U2 (AVDD) and U3 (VDDIO) switched on by ADIN_PWR"
- note removed: "${##}"
- note removed: "${#}"
- note removed: "${AUTHOR}"
- note removed: "${PCBPARTNUMBER}"
- note removed: "${REVISION}"
- note removed: "${TITLE}"
- moved on the sheet: D10, D8, D9, JP2, U1B
