File: nereus_Pi_shield_ADIN2111/BM_Mote_1_Load.kicad_sch (KiCad schematic)
At the start: 9 parts, among them U11 TPS26621DRCR

Commit message: S6.g: presentation clean-up (Nick's list) + active-low names (D30)
- Top-Level: VBUS_OUT beside the Load Switch; I2C page-long runs ->
  labelled stubs at the PoDL pins; R43 beside the ADIN HW_EN pin; J5
  spaced with its note
- Cover: mote renders + old index -> grey TBD box + real sheet index;
  dimensions TBD; revision table inside the page, about this board;
  licence note and CC logo clear of the title block
- ADIN: supplies and LED blocks spaced from U1A, with headers
- Power: 3V3 / 1V8 / 5V converters spaced, with headers
- All sheets: KiCad title block filled; Altium overlay texts removed
- Names: ~{ADIN_RST}, ~{ADIN_INT}, ~{ADIN_CS}, ~{ADIN_P1/P2_LED1},
  PAYLOAD_EN, ~{PAYLOAD_FAULT} (labels, hier labels, sheet pins)
- Same pin partition; ERC 495 -> 492 / 0 errors; 8 exclusion keys
  regenerated (reasons unchanged); netcheck 51/51; midwire 0
- Docs: DESIGN D30 + pin map, changelog, README, sofar_brief, TRACKER,
  viewer, DEV_LOG; schematic.pdf re-exported

Co-Authored-By: Claude Opus 5.5 <noreply@anthropic.com>
Connections:
- net SW_EN renamed PAYLOAD_EN
- net SW_FLAGB renamed ~{PAYLOAD_FAULT}
Other:
- note removed: "${##}"
- note removed: "${#}"
- note removed: "${AUTHOR}"
- note removed: "${PCBPARTNUMBER}"
- note removed: "${REVISION}"
- note removed: "${TITLE}"
Changed lines of the file:
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@@
 	(title_block
 		(title "Load Switch")
+		(date "2026-10-07")
 		(rev "AA")
-	)
-	(text "${##}"
-		(exclude_from_sim no)
-		(at 400.05 289.3822 0)
-		(effects
-			(font
-				(size 1.27 1.27)
-			)
-			(justify left bottom)
-		)
-	)
-	(text "${#}"
-		(exclude_from_sim no)
-		(at 395.224 289.3822 0)
-		(effects
-			(font
-				(size 1.27 1.27)
-			)
-			(justify left bottom)
-		)
-	)
-	(text "${PCBPARTNUMBER}"
-		(exclude_from_sim no)
-		(at 356.87 285.5722 0)
-		(effects
-			(font
-				(size 1.27 1.27)
-			)
-			(justify left bottom)
-		)
-	)
-	(text "${AUTHOR}"
-		(exclude_from_sim no)
-		(at 401.32 291.9222 0)
-		(effects
-			(font
-				(size 1.27 1.27)
-			)
-			(justify left bottom)
-		)
-	)
-	(text "${TITLE}"
-		(exclude_from_sim no)
-		(at 356.108 277.4442 0)
-		(effects
-			(font
-				(size 1.778 1.778)
-			)
-			(justify left bottom)
-		)
-	)
-	(text "${REVISION}"
-		(exclude_from_sim no)
-		(at 410.21 285.5722 0)
-		(effects
-			(font
-				(size 1.27 1.27)
-			)
-			(justify left bottom)
-		)
+		(comment 1 "${PCBPARTNAME} · ${PCBPARTNUMBER}")
+		(comment 2 "Author: ${AUTHOR}")
+		(comment 3 "Derived from Sofar Bristlemouth mote 000639-AB")
 	)
 	(text_box "Load Switch for VBUS"
@@
 		)
 	)
-	(label "SW_FLAGB"
+	(label "~{PAYLOAD_FAULT}"
 		(at 248.92 172.5422 0)
 		(effects
@@
 		)
 	)
-	(label "SW_ON"
+	(label "PAYLOAD_EN"
 		(at 199.39 154.7622 0)
 		(effects
@@
 		)
 	)
-	(hierarchical_label "SW_FLAGB"
+	(hierarchical_label "~{PAYLOAD_FAULT}"
 		(shape passive)
 		(at 281.94 172.5422 0)
@@
 		)
 	)
-	(hierarchical_label "SW_EN"
+	(hierarchical_label "PAYLOAD_EN"
 		(shape passive)
 		(at 129.54 172.5422 180)
