File: nereus_Pi_shield_ADIN2111/nereus_Pi_shield_ADIN2111.kicad_sch (KiCad schematic)
At the start: 0 parts

Commit message: S6.g: presentation clean-up (Nick's list) + active-low names (D30)
- Top-Level: VBUS_OUT beside the Load Switch; I2C page-long runs ->
  labelled stubs at the PoDL pins; R43 beside the ADIN HW_EN pin; J5
  spaced with its note
- Cover: mote renders + old index -> grey TBD box + real sheet index;
  dimensions TBD; revision table inside the page, about this board;
  licence note and CC logo clear of the title block
- ADIN: supplies and LED blocks spaced from U1A, with headers
- Power: 3V3 / 1V8 / 5V converters spaced, with headers
- All sheets: KiCad title block filled; Altium overlay texts removed
- Names: ~{ADIN_RST}, ~{ADIN_INT}, ~{ADIN_CS}, ~{ADIN_P1/P2_LED1},
  PAYLOAD_EN, ~{PAYLOAD_FAULT} (labels, hier labels, sheet pins)
- Same pin partition; ERC 495 -> 492 / 0 errors; 8 exclusion keys
  regenerated (reasons unchanged); netcheck 51/51; midwire 0
- Docs: DESIGN D30 + pin map, changelog, README, sofar_brief, TRACKER,
  viewer, DEV_LOG; schematic.pdf re-exported

Co-Authored-By: Claude Opus 5.5 <noreply@anthropic.com>
Other:
- note added: "1 Cover 2 Top-Level 3 ADIN2111 (Single-Pair Ethernet) 4 Load Switch (payload port) 5 PoDL (Power over Data Line) 6 Bus Power Monitor 7 Power (buck converters)"
- note added: "2026-10-07"
- note added: "First release, derived from Sofar mote 000639-AB"
- note added: "NB"
- note added: "Pi shield renders: TBD (after layout)"
- note added: "TBD (after layout)"
- note removed: "${##}"
- note removed: "${#}"
- note removed: "${AUTHOR}"
- note removed: "${REVISION}"
- note removed: "${TITLE}"
- note removed: "12/20/2023"
- note removed: "49 mm x 37 mm"
- note removed: "Adding silkscreen labels on BM ports ("1" and "2")"
- note removed: "BOTTOM VIEW"
- note removed: "SD + ES"
- note removed: "TOP VIEW"
