File: experiments/fable_layout_01/board/BM_Mote_1_Master.kicad_sch (KiCad schematic)
At the start: 34 parts, among them J1 Raspberry_Pi_2_3, J5 43650-0200

Commit message: fable layout 01 M0b: J5 stays the JST GH (Nick); schematic copy unchanged, board rebuilt
Co-Authored-By: Claude Fable 5.1 <noreply@anthropic.com>
Parts:
- J5: value 43650-0200 -> SM02B-GHS-TB; footprint Connector_Molex:Molex_Micro-Fit_3.0_43650-0200_1x02_P3.00mm_Horizontal -> Connector_JST:JST_GH_SM02B-GHS-TB_1x02-1MP_P1.25mm_Horizontal
Changed lines of the file:
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@@
 			)
 		)
-		(property "Value" "43650-0200"
+		(property "Value" "SM02B-GHS-TB"
 			(at 101.6 213.36 0)
 			(effects
@@
 			)
 		)
-		(property "Footprint" "Connector_Molex:Molex_Micro-Fit_3.0_43650-0200_1x02_P3.00mm_Horizontal"
+		(property "Footprint" "Connector_JST:JST_GH_SM02B-GHS-TB_1x02-1MP_P1.25mm_Horizontal"
 			(at 101.6 207.01 0)
 			(effects
