File: experiments/nick_raw_routing/nick_raw_routing.kicad_pcb (KiCad board)
At the start: 6 copper layers, 68 x 49 mm, 138 parts, among them J1 Raspberry_Pi_2_3, J2 Conn_02x12_Odd_Even, J5 SM02B-GHS-TB, T1 74930000, T2 74930000, U1 ADIN2111BCPZ, U10 LMR51430YDDCR, U11 TPS26621DRCR, U2 AP22913CN4-7, U3 AP22913CN4-7, U4 INA232AIDDFR, U5 LMR51430YDDCR, U6 TPS62840YBGR, Y1 ABM11W-25.0000MHZ-6-K1Z-T3

Commit message: Cleaned ERC before moving on to the Power 5V work
Parts:
- added J3: Conn_01x04, Connector_JST:JST_SH_SM04B-SRSS-TB_1x04-1MP_P1.00mm_Horizontal, F.Cu at (219.4, 36.6)
- added R10: RC0402JR-0710KL, Vault:FP-RC0402-0_4-IPC_C, F.Cu at (30.6, 17.9)
- added R24: RC0402JR-0710KL, Vault:FP-RC0402-0_4-IPC_C, F.Cu at (30.6, 20.4)
Connections:
- C13 pad 1: unconnected-(C13-Pad1) -> ADIN_VDDIO
- C14 pad 1: unconnected-(C14-Pad1) -> ADIN_VDDIO
- C49 pad 1: unconnected-(C49-Pad1) -> VBUS
- C5 pad 1: Net-(U1A-DLDO2_1P1) -> /Top-Level Schematic/ADIN/DVDD2_1P1
- C50 pad 1: unconnected-(C50-Pad1) -> VBUS_OUT
- C6 pad 1: unconnected-(C6-Pad1) -> /Top-Level Schematic/ADIN/DVDD1_1P1
- D3 pad 1: unconnected-(D3-C-Pad1) -> VBUS_OUT
- D4 pad 1: unconnected-(D4-Pad1) -> /Top-Level Schematic/BM1_P
- D5 pad 1: unconnected-(D5-Pad1) -> /Top-Level Schematic/BM2_P
- J1 pad 1: unconnected-(J1-3V3-Pad1)_1 -> PI_3V3
- J1 pad 17: unconnected-(J1-3V3-Pad1) -> PI_3V3
- J2 pad 1: unconnected-(J2-Pin_1-Pad1) -> /Top-Level Schematic/UART_TX
- J2 pad 10: unconnected-(J2-Pin_10-Pad10) -> GND
- J2 pad 11: unconnected-(J2-Pin_11-Pad11) -> PI_3V3
- J2 pad 12: unconnected-(J2-Pin_12-Pad12) -> GND
- J2 pad 13: unconnected-(J2-Pin_13-Pad13) -> /Top-Level Schematic/~{SPI0_CE1}
- J2 pad 14: unconnected-(J2-Pin_14-Pad14) -> GND
- J2 pad 15: unconnected-(J2-Pin_15-Pad15) -> /Top-Level Schematic/I2C0_SDA
- J2 pad 16: unconnected-(J2-Pin_16-Pad16) -> /Top-Level Schematic/I2C0_SCL
- J2 pad 17: unconnected-(J2-Pin_17-Pad17) -> /Top-Level Schematic/MOTOR_nSLEEP
- J2 pad 18: unconnected-(J2-Pin_18-Pad18) -> GND
- J2 pad 19: unconnected-(J2-Pin_19-Pad19) -> /Top-Level Schematic/MOTOR_IN1
- J2 pad 2: unconnected-(J2-Pin_2-Pad2) -> /Top-Level Schematic/~{ADC_ALERT}
- J2 pad 20: unconnected-(J2-Pin_20-Pad20) -> /Top-Level Schematic/MOTOR_IN2
- J2 pad 21: unconnected-(J2-Pin_21-Pad21) -> /Top-Level Schematic/SPI1_MISO
- J2 pad 22: unconnected-(J2-Pin_22-Pad22) -> /Top-Level Schematic/~{SPI1_CE2}
- J2 pad 23: unconnected-(J2-Pin_23-Pad23) -> /Top-Level Schematic/SPI1_SCLK
- J2 pad 24: unconnected-(J2-Pin_24-Pad24) -> /Top-Level Schematic/SPI1_MOSI
- J2 pad 3: unconnected-(J2-Pin_3-Pad3) -> /Top-Level Schematic/UART_RX
- J2 pad 4: unconnected-(J2-Pin_4-Pad4) -> GND
- J2 pad 5: unconnected-(J2-Pin_5-Pad5) -> /Top-Level Schematic/~{SPI1_CE0}
- J2 pad 6: unconnected-(J2-Pin_6-Pad6) -> /Top-Level Schematic/~{SPI1_CE1}
- J2 pad 7: unconnected-(J2-Pin_7-Pad7) -> /Top-Level Schematic/I2C3_SDA
- J2 pad 8: unconnected-(J2-Pin_8-Pad8) -> /Top-Level Schematic/I2C3_SCL
- J2 pad 9: unconnected-(J2-Pin_9-Pad9) -> PI_3V3
- R1 pad 1: unconnected-(R1-Pad1) -> /Top-Level Schematic/~{ADIN_INT}
- R8 pad 1: unconnected-(R8-Pad1) -> VBUS
- R8 pad 2: unconnected-(R8-Pad2) -> /Top-Level Schematic/PoDL/Power Monitor/P_IN
- TP13 pad 1: unconnected-(TP13-Pad1) -> /Top-Level Schematic/BM2_N
- TP20 pad 1: unconnected-(TP20-Pad1) -> 3V3
- TP21 pad 1: unconnected-(TP21-Pad1) -> 1V8
- TP22 pad 1: unconnected-(TP22-Pad1) -> VBUS
- TP3 pad 1: unconnected-(TP3-Pad1) -> /Top-Level Schematic/BM1_P
- TP36 pad 1: unconnected-(TP36-Pad1) -> VBUS_OUT
- TP38 pad 1: unconnected-(TP38-Pad1) -> /Top-Level Schematic/5V_PI
- TP5 pad 1: unconnected-(TP5-Pad1) -> /Top-Level Schematic/BM1_N
- TP7 pad 1: unconnected-(TP7-Pad1) -> /Top-Level Schematic/BM2_P
- U1 pad 14: Net-(U1A-DLDO2_1P1) -> /Top-Level Schematic/ADIN/DVDD2_1P1
- U1 pad 37: unconnected-(U1A-DLDO1_1P1-Pad37) -> /Top-Level Schematic/ADIN/DVDD1_1P1
