File: experiments/nick_raw_routing/nick_raw_routing.kicad_pcb (KiCad board)
At the start: 6 copper layers, 68 x 49 mm, 141 parts, among them J1 Raspberry_Pi_2_3, J2 Conn_02x12_Odd_Even, J3 Conn_01x04, J5 SM02B-GHS-TB, T1 74930000, T2 74930000, U1 ADIN2111BCPZ, U10 LMR51430YDDCR, U11 TPS26621DRCR, U2 AP22913CN4-7, U3 AP22913CN4-7, U4 INA232AIDDFR, U5 LMR51430YDDCR, U6 TPS62840YBGR, Y1 ABM11W-25.0000MHZ-6-K1Z-T3

Commit message: updates before the sofar review
Parts:
- added F1: Polyfuse, Fuse:Fuse_1206_3216Metric, F.Cu at (249.8, 55.1)
- added J4: Conn_01x02, Connector_JST:JST_PH_S2B-PH-K_1x02_P2.00mm_Horizontal, F.Cu at (246.5, 61.6)
- added J6: Connector_Generic:Conn_02x03_Odd_Even, Connector_PinHeader_2.54mm:PinHeader_2x03_P2.54mm_Vertical, F.Cu at (242.4, 75.1)
- JP1: value Bridged -> SolderJumper_3_Bridged12; footprint nereus:SolderJumper-2_R1210_Bridged_NetTie -> Jumper:SolderJumper-3_P1.3mm_Bridged12_RoundedPad1.0x1.5mm
- R15, R16: footprint Vault:CRCW08057R50FKEAHP-Footprint-1 -> Resistor_SMD:R_0805_2012Metric
- R34: footprint Vault:RESC1005X40X25LL05T10 -> Vault:FP-RC0402-0_4-IPC_C
- moved JP1 201.6 mm to (249.7, 51.1)
- moved D10 197.8 mm to (223.9, 35.3), turned to 90 degrees
- moved D8 193.1 mm to (220.4, 35.1), turned to 90 degrees
- moved D9 189.9 mm to (216.4, 35.1), turned to 90 degrees
- moved JP4 159.7 mm to (199.9, 76.4), turned to 90 degrees
- moved JP3 154.7 mm to (195.9, 76.4), turned to -90 degrees
- moved J5 147.4 mm to (188.9, 52.6), turned to -90 degrees
- moved J3 38.8 mm to (188.9, 60.6), turned to -90 degrees
- moved MP1 1.50 mm to (208.9, 36.1)
- moved MP2 1.50 mm to (199.4, 36.1)
- moved MP3 1.00 mm to (240.4, 36.1)
- moved MP4 1.00 mm to (230.9, 36.1)
- moved J2 0.74 mm to (232.7, 75.1)
