File: experiments/nick_raw_routing/BM_Mote_1_ADIN2111.kicad_sch (KiCad schematic)
At the start: 33 parts, among them U1 ADIN2111BCPZ, U2 AP22913CN4-7, U3 AP22913CN4-7, Y1 ABM11W-25.0000MHZ-6-K1Z-T3

Commit message: added straps
Parts:
- added JP3, JP4: SolderJumper_3_Bridged12, Jumper:SolderJumper-3_P1.3mm_Bridged12_RoundedPad1.0x1.5mm, symbol Jumper:SolderJumper_3_Bridged12
- added R9: ERJ-2RKF4701X, Vault:RESC1005X40X25LL05T05, symbol BM_Mote_000639-AB-altium-import:ADIN_0_RES-2_Altium Content Vault
Connections:
- net ADIN_VDDIO: now also JP3.1 (A), JP4.3 (B)
- net DVDD1_1P1: no longer U1.37 (DLDO1_1P1)
- net DVDD2_1P1: no longer U1.14 (DLDO2_1P1)
- net GND: now also JP3.3 (B), JP4.1 (A)
- new net CFG0_STRAP: JP4.2 (C)
- new net CFG1_STRAP: JP3.2 (C)
Other:
- note added: "CFG0_STRAP (pin43) defaults "0", cut trace and solder bridge to get "1""
- note added: "SPI_CFG1 (pin19) defaults "1" cut trace and solder bridge to get "0""
- moved on the sheet: D10, D8, D9, JP2, U1A, U1B, Y1

Commit message: Fix import connectivity
Connections:
- net DVDD1_1P1: now also U1.37 (DLDO1_1P1)
- net DVDD2_1P1: now also U1.14 (DLDO2_1P1)

Commit message: Cleaned ERC before moving on to the Power 5V work
Changed lines of the file:
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@@
 	)
 	(junction
+		(at 128.27 229.87)
+		(diameter 0)
+		(color 0 0 0 0)
+	)
+	(junction
 		(at 134.62 199.39)
 		(diameter 0)
@@
 	(wire
 		(pts
+			(xy 128.27 229.87) (xy 128.27 233.68)
+		)
+		(stroke
+			(width 0)
+			(type default)
+		)
+	)
+	(wire
+		(pts
 			(xy 78.74 196.85) (xy 71.12 196.85)
 		)
@@
 	(wire
 		(pts
+			(xy 128.27 229.87) (xy 144.78 229.87)
+		)
+		(stroke
+			(width 0)
+			(type default)
+		)
+	)
+	(wire
+		(pts
 			(xy 71.12 82.7278) (xy 77.47 82.7278)
 		)
@@
 	(wire
 		(pts
-			(xy 114.3 229.87) (xy 144.78 229.87)
+			(xy 114.3 229.87) (xy 128.27 229.87)
 		)
 		(stroke
@@
 					(unit 1)
 				)
+			)
+		)
+	)
+	(symbol
+		(lib_id "power:PWR_FLAG")
+		(at 128.27 233.68 180)
+		(unit 1)
+		(body_style 1)
+		(exclude_from_sim no)
+		(in_bom yes)
+		(on_board yes)
+		(in_pos_files yes)
+		(dnp no)
+		(property "Reference" "#FLG08"
+			(at 128.27 229.87 0)
+			(hide yes)
+			(show_name no)
+			(do_not_autoplace no)
+			(effects
+				(font
+					(size 1.27 1.27)
+				)
+			)
+		)
+		(property "Value" "PWR_FLAG"
+			(at 128.27 238.76 0)
+			(show_name no)
+			(do_not_autoplace no)
+			(effects
+				(font
+					(size 1.27 1.27)
+				)
+			)
+		)
+		(property "Footprint" ""
+			(at 128.27 233.68 0)
+			(hide yes)
+			(show_name no)
+			(do_not_autoplace no)
+			(effects
+				(font
+					(size 1.27 1.27)
+				)
+			)
+		)
+		(property "Datasheet" ""
+			(at 128.27 233.68 0)
+			(hide yes)
+			(show_name no)
+			(do_not_autoplace no)
+			(effects
+				(font
+					(size 1.27 1.27)
+				)
+			)
+		)
+		(property "Description" ""
+			(at 128.27 233.68 0)
+			(hide yes)
+			(show_name no)
+			(do_not_autoplace no)
+			(effects
+				(font
+					(size 1.27 1.27)
+				)
+			)
+		)
+		(pin "1"
+		)
+		(instances
+			(project "nick_raw_routing"
+				(path "/30e82bf5-1344-486b-817c-02d3b0649ce4/3c398828-e355-49f6-be37-cb3640d2c671/6b1c7de5-1c82-42d9-9a95-c340ffb1bf15"
+					(reference "#FLG08")
+					(unit 1)
+				)

Commit message: updates before the sofar review
Parts:
- U1: PLANNED LCSC (none) -> none shown yet; check My Parts; SOURCING JLC global sourcing (D26); no LCSC listing, DK 120 -> Bought: JLC global sourcing DOB202610190524705 (2026-10-18)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
- U2: SOURCING JLC global sourcing, all 40 (LCSC has 30) (D26) -> Bought: JLC global sourcing DOB202610190524705 (2026-10-18)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
- Y1: PLANNED LCSC (none) -> none shown yet; SOURCING JLC global sourcing (D26); no LCSC listing, DK 87 -> Bought: JLC global sourcing DOB202610190524705 (2026-10-18)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
Connections:
- net ADIN_AVDD: now also U2.A1 (VOUT)
- net AVDD_H + AVDD_L: now also U2.A2 (VIN)
- net GND: now also U2.B1 (GND)
- net HW_EN: now also U2.B2 (ON)
Changed lines of the file:
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@@
 			)
 		)
-		(property "SOURCING" "JLC global sourcing (D26); no LCSC listing, DK 120"
+		(property "SOURCING" "Bought: JLC global sourcing DOB202610190524705 (2026-10-18), qty 22, ready 2026-11-05"
 			(at 187.96 204.47 0)
 			(hide yes)
@@
 			)
 		)
-		(property "PLANNED LCSC" ""
+		(property "PLANNED LCSC" "none shown yet; check My Parts"
 			(at 187.96 204.47 0)
 			(hide yes)
@@
 			)
 		)
+		(property "Field12" ""
+			(at 187.96 204.47 0)
+			(hide yes)
+			(show_name no)
+			(do_not_autoplace no)
+			(effects
+				(font
+					(size 1.27 1.27)
+				)
+			)
+		)
 		(pin "2"
 		)
@@
 		(lib_id "BM_Mote_000639-AB-altium-import:ADIN_2_AP22913CN4-7-Symbol-1_Sofar Ocean Technologies, Inc.")
 		(at 106.68 199.39 0)
-		(unit 0)
+		(unit 1)
 		(body_style 1)
 		(exclude_from_sim no)
@@
 			)
 		)
-		(property "SOURCING" "JLC global sourcing, all 40 (LCSC has 30) (D26)"
+		(property "SOURCING" "Bought: JLC global sourcing DOB202610190524705 (2026-10-18), qty 42, ready 2026-11-05"
 			(at 106.68 199.39 0)
 			(hide yes)
@@
 				(path "/30e82bf5-1344-486b-817c-02d3b0649ce4/3c398828-e355-49f6-be37-cb3640d2c671/6b1c7de5-1c82-42d9-9a95-c340ffb1bf15"
 					(reference "U2")
-					(unit 0)
+					(unit 1)
 				)
 			)
@@
 			)
 		)
-		(property "SOURCING" "JLC global sourcing (D26); no LCSC listing, DK 120"
+		(property "SOURCING" "Bought: JLC global sourcing DOB202610190524705 (2026-10-18), qty 22, ready 2026-11-05"
 			(at 123.19 85.2678 0)
 			(hide yes)
@@
 			)
 		)
-		(property "PLANNED LCSC" ""
+		(property "PLANNED LCSC" "none shown yet; check My Parts"
 			(at 123.19 85.2678 0)
 			(hide yes)
@@
 			)
 		)
+		(property "Field12" ""
+			(at 123.19 85.2678 0)
+			(hide yes)
+			(show_name no)
+			(do_not_autoplace no)
+			(effects
+				(font
+					(size 1.27 1.27)
+				)
+			)
+		)
 		(pin "48"
 		)
@@
 			)
 		)
-		(property "SOURCING" "JLC global sourcing (D26); no LCSC listing, DK 87"
+		(property "SOURCING" "Bought: JLC global sourcing DOB202610190524705 (2026-10-18), qty 22, ready 2026-11-05"
 			(at 176.53 118.11 0)
 			(hide yes)
@@
 			)
 		)
-		(property "PLANNED LCSC" ""
+		(property "PLANNED LCSC" "none shown yet"
 			(at 176.53 118.11 0)
 			(hide yes)
