File: experiments/nick_raw_routing/BM_Mote_1_Master.kicad_sch (KiCad schematic)
At the start: 34 parts, among them J1 Raspberry_Pi_2_3, J5 SM02B-GHS-TB

Commit message: Added I2C0, I2C1, I2C2 and fix to load switch
Parts:
- added J2: Conn_02x12_Odd_Even, Connector_PinHeader_2.54mm:PinHeader_2x12_P2.54mm_Vertical, symbol Connector_Generic:Conn_02x12_Odd_Even
Connections:
- net PAYLOAD_EN: now also J1.37 (GPIO26); no longer J1.36 (GPIO16)
- net ~{PAYLOAD_FAULT}: now also J1.31 (GCLK2/GPIO6); no longer J1.38 (GPIO20/MOSI1)
- net UART_RX: now reaches J1.10 (GPIO15/RXD)
- net ~{SPI1_CE1}: now reaches J1.11 (GPIO17)
- net ~{SPI1_CE0}: now reaches J1.12 (GPIO18/PWM0)
- net I2C3_SCL: now reaches J1.13 (GPIO27)
- net I2C3_SDA: now reaches J1.15 (GPIO22)
- net ~{SPI0_CE1}: now reaches J1.26 (~{CE1}/GPIO7)
- net I2C0_SDA: now reaches J1.27 (ID_SD/GPIO0)
- net I2C0_SCL: now reaches J1.28 (ID_SC/GPIO1)
- net MOTOR_nSLEEP: now reaches J1.29 (GCLK1/GPIO5)
- net MOTOR_IN1: now reaches J1.32 (PWM0/GPIO12)
- net MOTOR_IN2: now reaches J1.33 (PWM1/GPIO13)
- net SPI1_MISO: now reaches J1.35 (GPIO19/MISO1)
- net SPI1_SCLK: now reaches J1.40 (GPIO21/SCLK1)
- net ~{ADC_ALERT}: now reaches J1.7 (GCLK0/GPIO4)
- net UART_TX: now reaches J1.8 (GPIO14/TXD)
- net I2C1_SCL: no longer names the net of J1.5 (SCL/GPIO3)
- net I2C1_SDA: no longer names the net of J1.3 (SDA/GPIO2)
- new net SPI1_MOSI: J1.38 (GPIO20/MOSI1)
- new net ~{SPI1_CE2}: J1.36 (GPIO16)
- no-connect marks 18 -> 3

Commit message: Fix import connectivity
Parts:
- added J3: Conn_01x04, Connector_JST:JST_SH_SM04B-SRSS-TB_1x04-1MP_P1.00mm_Horizontal, symbol Connector_Generic:Conn_01x04
- added R10, R24: RC0402JR-0710KL, Vault:FP-RC0402-0_4-IPC_C, symbol BM_Mote_000639-AB-altium-import:P1_3_1029c3af85768c4190bb7ad29bc67b5_Altium Con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
Connections:
- net GND: now also J2.10 (Pin_10), J2.12 (Pin_12), J2.14 (Pin_14), J2.18 (Pin_18), J2.4 (Pin_4), J3.1 (Pin_1)
- net I2C0_SCL: now also J2.16 (Pin_16)
- net I2C0_SDA: now also J2.15 (Pin_15)
- net I2C3_SCL: now also J2.8 (Pin_8), J3.4 (Pin_4)
- net I2C3_SDA: now also J2.7 (Pin_7), J3.3 (Pin_3)
- net MOTOR_IN1: now also J2.19 (Pin_19)
- net MOTOR_IN2: now also J2.20 (Pin_20)
- net MOTOR_nSLEEP: now also J2.17 (Pin_17)
- net SPI1_MISO: now also J2.21 (Pin_21)
- net SPI1_MOSI: now also J2.24 (Pin_24)
- net SPI1_SCLK: now also J2.23 (Pin_23)
- net UART_RX: now also J2.3 (Pin_3)
- net UART_TX: now also J2.1 (Pin_1)
- net ~{ADC_ALERT}: now also J2.2 (Pin_2)
- net ~{SPI0_CE1}: now also J2.13 (Pin_13)
- net ~{SPI1_CE0}: now also J2.5 (Pin_5)
- net ~{SPI1_CE1}: now also J2.6 (Pin_6)
- net ~{SPI1_CE2}: now also J2.22 (Pin_22)
- net PI_3V3: now reaches J2.11 (Pin_11)
- net PI_3V3: now also J1.1 (3V3), J1.17 (3V3), J2.9 (Pin_9), J3.2 (Pin_2)
- no-connect marks 3 -> 2
Other:
- note added: "I2C1 GPIO2/3 = LiFePO4wered only (0x43). Pi's 1.8k pull-ups. I2C0 GPIO0/1 = shield: INA232 0x41, ADS1115 0x48 (bluewired). R26/R27 4.7k to PI_3V3. Keep 0x50 free (HAT EEPROM probe at boot). I2C3 GPIO22/27 = software I2C, Qwiic. Qwiic power and pull-ups on PI_3V3. J2 breakout 3V3 pins (9, 11) = PI_3V3. Shield 3V3 is for shield parts only. ADS1115: AIN0 = MP6550 VISEN (200 mV/A), AIN1 = shaft pot, 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"

Commit message: Cleaned ERC before moving on to the Power 5V work
Connections:
- no-connect marks 2 -> 6

Commit message: updates before the sofar review
Parts:
- removed JP1: Bridged, nereus:SolderJumper-2_R1210_Bridged_NetTie, symbol Jumper:SolderJumper_2_Bridged
- added F1: Polyfuse, Fuse:Fuse_1206_3216Metric, symbol Device:Polyfuse
- added J4: Conn_01x02, Connector_JST:JST_PH_S2B-PH-K_1x02_P2.00mm_Horizontal, symbol Connector_Generic:Conn_01x02
- added J6: PI 3V3 header (DNP), Connector_PinHeader_2.54mm:PinHeader_2x03_P2.54mm_Vertical, symbol Connector_Generic:Conn_02x03_Odd_Even
- added JP1: SolderJumper_3_Bridged12, Jumper:SolderJumper-3_P1.3mm_Bridged12_RoundedPad1.0x1.5mm, symbol Jumper:SolderJumper_3_Bridged12
- J2: Planned Note (none) -> DNP: dev/bluewire pads; hand-fit 2.54 mm header if needed; now not fitted; now left out of the parts list
- J3: value Conn_01x04 -> Con. 1x04; Planned LCSC (none) -> C160404
- J5: SOURCING JLC global sourcing (D26); LCSC C189893 out of stock, DK 10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 -> JLC Parts
- MP1: PLANNED LCSC (none) -> C17256375; SOURCING JLC global sourcing (D26); no LCSC listing, DK 7,835 -> Bought: JLC global sourcing DOB202610190524705 (2026-10-18)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
Connections:
- net 5V_PI: now also JP1.2 (C)
- net BM1_P: now also MP1.1
- net GND: now also J4.2 (Pin_2), J6.2 (Pin_2), J6.4 (Pin_4), J6.6 (Pin_6)
- net PI_3V3: now also J6.1 (Pin_1), J6.3 (Pin_3), J6.5 (Pin_5)
- net PI_5V: now also JP1.1 (A)
- new net: F1.2, J4.1 (Pin_1)
- new net 5V_LIFEPO4: F1.1, JP1.3 (B)
Other:
- note added: "JP1 power mode (middle pad = shield 5V, 5V_PI): Mode 1 (as built): pads 1-2 bridged -> shield powers the Pi through J1 pin 2. Mode 2 (LiFePO4wered): cut 1-2, bridge 2-3 -> shield 5V goes out on the JST-PH to the LiFePO4wered INPUT. Never wire it to the LiFePO4wered 5V output. Never plug a 5 V source into the Pi's USB while 1-2 is bridged."
- note removed: "JP1 bridged as built: the shield powers the Pi (D14). Bridged: never plug a 5 V source into the Pi's USB (charger, PC, self-powered hub), shield powered or not. USB peripherals powered by the Pi are OK. Pi powered elsewhere (battery pack): cut the bridge before potting; refit a 0R 1210 (CRCW12100000Z0EA) to reconnect."
- moved on the sheet: J1, J3, J5
