File: experiments/nick_raw_routing/BM_Mote_1_PoDL.kicad_sch (KiCad schematic)
At the start: 28 parts, among them T1 74930000, T2 74930000

Commit message: added straps
Parts:
- R15, R16: footprint Vault:CRCW08057R50FKEAHP-Footprint-1 -> 0805; FOOTPRINT 0805 -> (none)

Commit message: Cleaned ERC before moving on to the Power 5V work
Parts:
- R15, R16: footprint 0805 -> Resistor_SMD:R_0805_2012Metric
Connections:
- net VBUS: now also R15.2, R16.2
Changed lines of the file:
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@@
 		(lib_id "BM_Mote_000639-AB-altium-import:PODL_1_CRCW08057R50FKEAHP_Sofar Ocean Technologies, Inc.")
 		(at 335.28 134.4422 0)
-		(unit 0)
+		(unit 1)
 		(body_style 1)
 		(exclude_from_sim no)
@@
 			)
 		)
-		(property "Footprint" "0805"
+		(property "Footprint" "Resistor_SMD:R_0805_2012Metric"
 			(at 336.042 141.8082 0)
+			(hide yes)
 			(show_name no)
 			(do_not_autoplace no)
@@
 				(path "/30e82bf5-1344-486b-817c-02d3b0649ce4/3c398828-e355-49f6-be37-cb3640d2c671/a31c5b59-6e77-4130-b11e-1392851c8b62"
 					(reference "R16")
-					(unit 0)
+					(unit 1)
 				)
 			)
@@
 		(lib_id "BM_Mote_000639-AB-altium-import:PODL_1_CRCW08057R50FKEAHP_Sofar Ocean Technologies, Inc.")
 		(at 312.42 134.4422 0)
-		(unit 0)
+		(unit 1)
 		(body_style 1)
 		(exclude_from_sim no)
@@
 			)
 		)
-		(property "Footprint" "0805"
+		(property "Footprint" "Resistor_SMD:R_0805_2012Metric"
 			(at 313.182 141.8082 0)
+			(hide yes)
 			(show_name no)
 			(do_not_autoplace no)
@@
 				(path "/30e82bf5-1344-486b-817c-02d3b0649ce4/3c398828-e355-49f6-be37-cb3640d2c671/a31c5b59-6e77-4130-b11e-1392851c8b62"
 					(reference "R15")
-					(unit 0)
+					(unit 1)
 				)
 			)

Commit message: updates before the sofar review
Parts:
- C22: ALT NOTE Sofar review: bus damping; a newly sourced replacement must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 -> (none); PLANNED NOTE As specified (Sofar review): no potting-safe like-for-like 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 -> (none); SOURCING JLC global sourcing (first build) until an ALT is approved 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 -> JLC global sourcing (first build)
- D1: PLANNED NOTE Sofar's own listed second source (their MANUFACTURERPARTNUMBER1); ST SMA6F33A is obsolete (DK); no LCSC listing found (2026-10-06): JLC global sourcing; Sofar Q7 -> Sofar's own listed second source (their MANUFACTURERPARTNUMBER1); SOURCING JLC global sourcing of Sofar's second source Vishay SMA6F33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 -> Bought: JLC global sourcing DOB202610190524705 (2026-10-18)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
- D2: PLANNED LCSC (none) -> C3757753; SOURCING JLC global sourcing (D26); no LCSC listing -> Bought: JLC global sourcing DOB202610190524705 (2026-10-18)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
- R12, R13, R17, R19: now not fitted; now left out of the parts list
- R15: ALT NOTE Sofar review: 7.5 Ω ±1 % 0.5 W, ±200 vs ±100 ppm/°C, pulse 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 -> (none); ALT1 LCSC C873769 -> (none); ALT1 MFR YAGEO -> (none); ALT1 MPN SR0805FR-477R5L -> (none); PLANNED LCSC (none) -> wait for JLC update; PLANNED NOTE As specified (Sofar review): the only stocked alternate (YA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 -> (none); SOURCING JLC global sourcing (first build) until an ALT is approved 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 -> JLC global sourcing (first build)
Connections:
- net BM1_N: now also R13.2
- net BM1_P: now also R12.1
- net BM2_N: now also R19.2
- net BM2_P: now also R17.1
- net GND: now also C22.1 (C), D1.1 (ANODE), D2.2 (A), R13.1, R19.1
- net Power Monitor/P_IN: now also R17.2
- net VBUS: now also D1.2 (CATHODE), D2.1 (C), R12.2
- net at R15.1: now also C22.2 (A)
Changed lines of the file:
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@@
 		(lib_id "BM_Mote_000639-AB-altium-import:PODL_2_1029c3af85768c4190bb7ad29bc67b5_Altium Content Vault")
 		(at 256.54 103.9622 0)
-		(unit 0)
+		(unit 1)
 		(body_style 1)
 		(exclude_from_sim no)
-		(in_bom yes)
+		(in_bom no)
 		(on_board yes)
 		(in_pos_files yes)
-		(dnp no)
+		(dnp yes)
 		(property "Reference" "R13"
 			(at 242.824 102.4382 0)
@@
 				(path "/30e82bf5-1344-486b-817c-02d3b0649ce4/3c398828-e355-49f6-be37-cb3640d2c671/a31c5b59-6e77-4130-b11e-1392851c8b62"
 					(reference "R13")
-					(unit 0)
+					(unit 1)
 				)
 			)
@@
 		(lib_id "BM_Mote_000639-AB-altium-import:PODL_0_a00bbbee19879c290e62620ae7e47b1_Altium Content Vault")
 		(at 312.42 147.1422 0)
-		(unit 0)
+		(unit 1)
 		(body_style 1)
 		(exclude_from_sim no)
@@
 			)
 		)
-		(property "ALT NOTE" "Sofar review: bus damping; a newly sourced replacement must be potting-safe (constraint 8), so no like-for-like alternate; JLC global sourcing"
+		(property "ALT NOTE" ""
 			(at 312.42 147.1422 0)
 			(hide yes)
@@
 			)
 		)
-		(property "SOURCING" "JLC global sourcing (first build) until an ALT is approved (D26)"
+		(property "SOURCING" "JLC global sourcing (first build) "
 			(at 312.42 147.1422 0)
 			(hide yes)
@@
 			)
 		)
-		(property "PLANNED NOTE" "As specified (Sofar review): no potting-safe like-for-like alternate (constraint 8); LCSC listing out of stock: JLC global sourcing"
+		(property "PLANNED NOTE" ""
 			(at 312.42 147.1422 0)
 			(hide yes)
@@
 				(path "/30e82bf5-1344-486b-817c-02d3b0649ce4/3c398828-e355-49f6-be37-cb3640d2c671/a31c5b59-6e77-4130-b11e-1392851c8b62"
 					(reference "C22")
-					(unit 0)
+					(unit 1)
 				)
 			)
@@
 		(lib_id "BM_Mote_000639-AB-altium-import:PODL_2_1029c3af85768c4190bb7ad29bc67b5_Altium Content Vault")
 		(at 256.54 73.4822 0)
-		(unit 0)
+		(unit 1)
 		(body_style 1)
 		(exclude_from_sim no)
-		(in_bom yes)
+		(in_bom no)
 		(on_board yes)
 		(in_pos_files yes)
-		(dnp no)
+		(dnp yes)
 		(property "Reference" "R12"
 			(at 242.824 71.9582 0)
@@
 				(path "/30e82bf5-1344-486b-817c-02d3b0649ce4/3c398828-e355-49f6-be37-cb3640d2c671/a31c5b59-6e77-4130-b11e-1392851c8b62"
 					(reference "R12")
-					(unit 0)
+					(unit 1)
 				)
 			)
@@
 		(lib_id "BM_Mote_000639-AB-altium-import:PODL_2_1029c3af85768c4190bb7ad29bc67b5_Altium Content Vault")
 		(at 256.54 208.1022 0)
-		(unit 0)
+		(unit 1)
 		(body_style 1)
 		(exclude_from_sim no)
-		(in_bom yes)
+		(in_bom no)
 		(on_board yes)
 		(in_pos_files yes)
-		(dnp no)
+		(dnp yes)
 		(property "Reference" "R17"
 			(at 242.824 206.5782 0)
@@
 				(path "/30e82bf5-1344-486b-817c-02d3b0649ce4/3c398828-e355-49f6-be37-cb3640d2c671/a31c5b59-6e77-4130-b11e-1392851c8b62"
 					(reference "R17")
-					(unit 0)
+					(unit 1)
 				)
 			)
@@
 			)
 		)
-		(property "ALT1 MPN" "SR0805FR-477R5L"
+		(property "ALT1 MPN" ""
 			(at 312.42 134.4422 0)
 			(hide yes)
@@
 			)
 		)
-		(property "ALT1 MFR" "YAGEO"
+		(property "ALT1 MFR" ""
 			(at 312.42 134.4422 0)
 			(hide yes)
@@
 			)
 		)
-		(property "ALT1 LCSC" "C873769"
+		(property "ALT1 LCSC" ""
 			(at 312.42 134.4422 0)
 			(hide yes)
@@
 			)
 		)
-		(property "ALT NOTE" "Sofar review: 7.5 Ω ±1 % 0.5 W, ±200 vs ±100 ppm/°C, pulse rating not stated"
+		(property "ALT NOTE" ""
 			(at 312.42 134.4422 0)
 			(hide yes)
@@
 			)
 		)
-		(property "SOURCING" "JLC global sourcing (first build) until an ALT is approved (D26)"
+		(property "SOURCING" "JLC global sourcing (first build) "
 			(at 312.42 134.4422 0)
 			(hide yes)
@@
 			)
 		)
-		(property "PLANNED LCSC" ""
+		(property "PLANNED LCSC" "wait for JLC update"
 			(at 312.42 134.4422 0)
 			(hide yes)
@@
 			)
 		)
-		(property "PLANNED NOTE" "As specified (Sofar review): the only stocked alternate (YAGEO SR0805, ALT1) has no stated pulse rating and ±200 vs ±100 ppm/°C; JLC global sourcing: no LCSC listing"
+		(property "PLANNED NOTE" ""
 			(at 312.42 134.4422 0)
 			(hide yes)
@@
 		(lib_id "BM_Mote_000639-AB-altium-import:PODL_1_c1678fac7984e62e0809fbf79c06691_Sofar Ocean Technologies, Inc.")
 		(at 383.54 152.2222 0)
-		(unit 0)
+		(unit 1)
 		(body_style 1)
 		(exclude_from_sim no)
@@
 			)
 		)
-		(property "SOURCING" "JLC global sourcing (D26); no LCSC listing"
+		(property "SOURCING" "Bought: JLC global sourcing DOB202610190524705 (2026-10-18), qty 45, ready 2026-11-05"
 			(at 383.54 152.2222 0)
 			(hide yes)
@@
 			)
 		)
-		(property "PLANNED LCSC" ""
+		(property "PLANNED LCSC" "C3757753"
 			(at 383.54 152.2222 0)
 			(hide yes)
@@
 				(path "/30e82bf5-1344-486b-817c-02d3b0649ce4/3c398828-e355-49f6-be37-cb3640d2c671/a31c5b59-6e77-4130-b11e-1392851c8b62"
 					(reference "D2")
-					(unit 0)
+					(unit 1)
 				)
 			)
@@
 		(lib_id "BM_Mote_000639-AB-altium-import:PODL_2_1029c3af85768c4190bb7ad29bc67b5_Altium Content Vault")
 		(at 256.54 238.5822 0)
-		(unit 0)
+		(unit 1)
 		(body_style 1)
 		(exclude_from_sim no)
-		(in_bom yes)
+		(in_bom no)
 		(on_board yes)
 		(in_pos_files yes)
-		(dnp no)
+		(dnp yes)
 		(property "Reference" "R19"
 			(at 242.824 237.0582 0)
@@
 				(path "/30e82bf5-1344-486b-817c-02d3b0649ce4/3c398828-e355-49f6-be37-cb3640d2c671/a31c5b59-6e77-4130-b11e-1392851c8b62"
 					(reference "R19")
-					(unit 0)
+					(unit 1)
 				)
 			)
@@
 		(lib_id "BM_Mote_000639-AB-altium-import:PODL_1_SMA6F33A_Sofar Ocean Technologies, Inc.")
 		(at 358.14 144.6022 0)
-		(unit 0)
+		(unit 1)
 		(body_style 1)
 		(exclude_from_sim no)
@@
 			)
 		)
-		(property "SOURCING" "JLC global sourcing of Sofar's second source Vishay SMA6F33A-M3/H (ST part obsolete; Sofar Q7) (D26)"
+		(property "SOURCING" "Bought: JLC global sourcing DOB202610190524705 (2026-10-18), qty 27, ready 2026-11-05"
 			(at 358.14 144.6022 0)
 			(hide yes)
@@
 			)
 		)
-		(property "PLANNED NOTE" "Sofar's own listed second source (their MANUFACTURERPARTNUMBER1); ST SMA6F33A is obsolete (DK); no LCSC listing found (2026-10-06): JLC global sourcing; Sofar Q7"
+		(property "PLANNED NOTE" "Sofar's own listed second source (their MANUFACTURERPARTNUMBER1)"
 			(at 358.14 144.6022 0)
 			(hide yes)
@@
 				(path "/30e82bf5-1344-486b-817c-02d3b0649ce4/3c398828-e355-49f6-be37-cb3640d2c671/a31c5b59-6e77-4130-b11e-1392851c8b62"
 					(reference "D1")
-					(unit 0)
+					(unit 1)
 				)
 			)
