File: experiments/nick_raw_routing/BM_Mote_1_Power.kicad_sch (KiCad schematic)
At the start: 26 parts, among them U10 LMR51430YDDCR, U5 LMR51430YDDCR, U6 TPS62840YBGR

Commit message: Fix import connectivity
Changed lines of the file:
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@@
 	)
 	(junction
+		(at 177.8 78.5622)
+		(diameter 0)
+		(color 0 0 0 0)
+	)
+	(junction
 		(at 95.25 215.7222)
 		(diameter 0)
@@
 	)
 	(junction
+		(at 172.72 78.5622)
+		(diameter 0)
+		(color 0 0 0 0)
+	)
+	(junction
 		(at 74.93 239.8522)
 		(diameter 0)
@@
 	(wire
 		(pts
+			(xy 177.8 78.5622) (xy 177.8 78.74)
+		)
+		(stroke
+			(width 0)
+			(type default)
+		)
+	)
+	(wire
+		(pts
 			(xy 181.61 220.8022) (xy 187.96 220.8022)
 		)
@@
 	(wire
 		(pts
+			(xy 172.72 77.47) (xy 172.72 78.5622)
+		)
+		(stroke
+			(width 0)
+			(type default)
+		)
+	)
+	(wire
+		(pts
 			(xy 205.74 97.6122) (xy 205.74 95.0722)
 		)
@@
 	(wire
 		(pts
+			(xy 172.72 78.5622) (xy 172.72 78.74)
+		)
+		(stroke
+			(width 0)
+			(type default)
+		)
+	)
+	(wire
+		(pts
+			(xy 177.8 77.47) (xy 177.8 78.5622)
+		)
+		(stroke
+			(width 0)
+			(type default)
+		)
+	)
+	(wire
+		(pts
 			(xy 128.27 225.8822) (xy 125.73 225.8822)
 		)
@@
 	(symbol
 		(lib_id "BM_Mote_000639-AB-altium-import:POWER_3_b4654b650e69147ec39a6b967a45e02_Altium Content Vault")
-		(at 177.8 78.5622 0)
+		(at 177.8 77.47 0)
 		(unit 0)
 		(body_style 1)
@@
 		(dnp no)
 		(property "Reference" "C28"
-			(at 173.736 75.7682 0)
+			(at 173.736 74.676 0)
 			(show_name no)
 			(do_not_autoplace no)
@@
 		)
 		(property "Value" "CL05A104KA5NNNC"
-			(at 172.212 75.7682 0)
+			(at 172.212 74.676 0)
 			(hide yes)
 			(show_name no)
@@
 		)
 		(property "Footprint" "Vault:FP-CL278-IPC_C"
-			(at 177.8 78.5622 0)
+			(at 177.8 77.47 0)
 			(hide yes)
 			(show_name no)
@@
 		)
 		(property "Datasheet" ""
-			(at 177.8 78.5622 0)
+			(at 177.8 77.47 0)
 			(hide yes)
 			(show_name no)
@@
 		)
 		(property "Description" "Cap Ceramic 100nF 25V X5R ±10% SMD 0402 +85°C Paper T/R"
-			(at 177.8 78.5622 0)
+			(at 177.8 77.47 0)
 			(hide yes)
 			(show_name no)
@@
 		)
 		(property "PACKAGE QUANTITY" "1"
-			(at 172.212 75.7682 0)
+			(at 172.212 74.676 0)
 			(hide yes)
 			(show_name no)
@@
 		)
 		(property "HEIGHT" "0.5mm"
-			(at 172.212 75.7682 0)
+			(at 172.212 74.676 0)
 			(hide yes)
 			(show_name no)
@@
 		)
 		(property "CASE CODE (METRIC)" "1005"
-			(at 172.212 75.7682 0)
+			(at 172.212 74.676 0)
 			(hide yes)
 			(show_name no)
@@
 		)
 		(property "THICKNESS" "0.022inch"
-			(at 172.212 75.7682 0)
+			(at 172.212 74.676 0)
 			(hide yes)
 			(show_name no)
@@
 		)
 		(property "MOUNT" "Surface Mount"
-			(at 172.212 75.7682 0)
+			(at 172.212 74.676 0)
 			(hide yes)
 			(show_name no)
@@
 		)
 		(property "LEAD FREE" "Lead Free"
-			(at 172.212 75.7682 0)
+			(at 172.212 74.676 0)
 			(hide yes)
 			(show_name no)
@@
 		)
 		(property "CASE CODE (IMPERIAL)" "0402"
-			(at 177.8 73.4822 0)
+			(at 177.8 72.39 0)
 			(show_name no)
 			(do_not_autoplace no)
@@
 		)
 		(property "PACKAGING" "Tape and Reel"
-			(at 172.212 75.7682 0)
+			(at 172.212 74.676 0)
 			(hide yes)
 			(show_name no)
@@
 		)
 		(property "DEPTH" "0.5mm"
-			(at 172.212 75.7682 0)
+			(at 172.212 74.676 0)
 			(hide yes)
 			(show_name no)
@@
 		)
 		(property "VOLTAGE" "25V"
-			(at 172.72 73.4822 0)
+			(at 172.72 72.39 0)
 			(show_name no)
 			(do_not_autoplace no)
@@
 		)
 		(property "MIN OPERATING TEMPERATURE" "-55°C"
-			(at 172.212 75.7682 0)
+			(at 172.212 74.676 0)
 			(hide yes)
 			(show_name no)
@@
 		)
 		(property "VOLTAGE RATING" "25V"
-			(at 172.212 75.7682 0)
+			(at 172.212 74.676 0)
 			(hide yes)
 			(show_name no)
@@
 		)
 		(property "DIELECTRIC" "X5R"
-			(at 172.212 75.7682 0)
+			(at 172.212 74.676 0)
 			(hide yes)
 			(show_name no)
@@
 		)
 		(property "CASE/PACKAGE" "0402"
-			(at 172.212 75.7682 0)
+			(at 172.212 74.676 0)
 			(hide yes)
 			(show_name no)
@@
 		)
 		(property "TOLERANCE" "10%"
-			(at 172.212 75.7682 0)
+			(at 172.212 74.676 0)
 			(hide yes)
 			(show_name no)
@@
 		)
 		(property "WIDTH" "0.02inch"
-			(at 172.212 75.7682 0)
+			(at 172.212 74.676 0)
 			(hide yes)
 			(show_name no)
@@
 		)
 		(property "MAX OPERATING TEMPERATURE" "85°C"
-			(at 172.212 75.7682 0)
+			(at 172.212 74.676 0)
 			(hide yes)
 			(show_name no)
@@
 		)
 		(property "CAPACITANCE" "100nF"
-			(at 172.466 71.4502 0)
+			(at 172.466 70.358 0)
 			(show_name no)
 			(do_not_autoplace no)
@@
 		)
 		(property "LENGTH" "1mm"
-			(at 172.212 75.7682 0)
+			(at 172.212 74.676 0)
 			(hide yes)
 			(show_name no)
@@
 		)
 		(property "RADIATION HARDENING" "No"
-			(at 172.212 75.7682 0)
+			(at 172.212 74.676 0)
 			(hide yes)
 			(show_name no)
@@
 		)
 		(property "VOLTAGE RATING (DC)" "25V"
-			(at 172.212 75.7682 0)
+			(at 172.212 74.676 0)
 			(hide yes)
 			(show_name no)
@@
 		)
 		(property "SHEET" "ADIN2111"
-			(at 172.212 75.7682 0)
+			(at 172.212 74.676 0)
 			(hide yes)
 			(show_name no)
@@
 		)
 		(property "PLANNED MPN" "CL05A104KA5NNNC"
-			(at 177.8 78.5622 0)
+			(at 177.8 77.47 0)
 			(hide yes)
 			(show_name no)
@@
 		)
 		(property "PLANNED MFR" "Samsung"
-			(at 177.8 78.5622 0)
+			(at 177.8 77.47 0)
 			(hide yes)
 			(show_name no)
@@
 		)
 		(property "PLANNED LCSC" "C100072"
-			(at 177.8 78.5622 0)
+			(at 177.8 77.47 0)
 			(hide yes)
 			(show_name no)
@@
 		)
 		(property "PLANNED NOTE" "As specified; in LCSC stock (checked 2026-10-06)"
-			(at 177.8 78.5622 0)
+			(at 177.8 77.47 0)
 			(hide yes)
 			(show_name no)
@@
 		)
 		(property "MANUFACTURER" "Samsung"
-			(at 177.8 78.5622 0)
+			(at 177.8 77.47 0)
 			(hide yes)
 			(show_name no)

Commit message: updates before the sofar review
Parts:
- L3: PLANNED LCSC (none) -> none shown yet; SOURCING JLC global sourcing (D26); no LCSC listing -> Bought: JLC global sourcing DOB202610190524705 (2026-10-18)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
- R38: value RC0402FR-0713K7L -> 0402WGF1332TCE; MANUFACTURER Yageo -> UNI-ROYAL; PLANNED LCSC C274888 -> C122547; PLANNED MFR Yageo -> UNI-ROYAL; PLANNED MPN RC0402FR-0713K7L -> 0402WGF1332TCE; PLANNED NOTE As specified; in LCSC stock (checked 2026-10-06) -> 13.3k 1% 0402 for 5V buck at 5.11 V (was 13.7k); same UNI-R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; RESISTANCE 13.7kR -> 13.3kR
Connections:
- net 3V3: now also L3.2
- net 3V3_Buck_SW: now also L3.1
- net 5V_FB: now also R38.1
- net GND: now also R38.2
Other:
- note added: "5V_PI = 0.6 V × (1 + 100k/13.3k) = 5.11 V"
Changed lines of the file:
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@@
 		)
 	)
+	(text "5V_PI = 0.6 V × (1 + 100k/13.3k) = 5.11 V"
+		(exclude_from_sim no)
+		(at 203.2 260.604 0)
+		(effects
+			(font
+				(size 1.27 1.27)
+			)
+		)
+	)
 	(junction
 		(at 254 220.8022)
@@
 		(lib_id "BM_Mote_000639-AB-altium-import:POWER_0_725321dda6339637d4d059423bc1c3c_Sofar Ocean Technologies, Inc.")
 		(at 187.96 83.6422 0)
-		(unit 0)
+		(unit 1)
 		(body_style 1)
 		(exclude_from_sim no)
@@
 			)
 		)
-		(property "SOURCING" "JLC global sourcing (D26); no LCSC listing"
+		(property "SOURCING" "Bought: JLC global sourcing DOB202610190524705 (2026-10-18), qty 42, ready 2026-11-05"
 			(at 187.96 83.6422 0)
 			(hide yes)
@@
 			)
 		)
-		(property "PLANNED LCSC" ""
+		(property "PLANNED LCSC" "none shown yet"
 			(at 187.96 83.6422 0)
 			(hide yes)
@@
 				(path "/30e82bf5-1344-486b-817c-02d3b0649ce4/3c398828-e355-49f6-be37-cb3640d2c671/4eeafcb7-a684-4b4d-adeb-0d10d663bf3a"
 					(reference "L3")
-					(unit 0)
+					(unit 1)
 				)
 			)
@@
 		(lib_id "BM_Mote_000639-AB-altium-import:POWER_3_1029c3af85768c4190bb7ad29bc67b5_Altium Content Vault")
 		(at 232.41 251.2822 0)
-		(unit 0)
+		(unit 1)
 		(body_style 1)
 		(exclude_from_sim no)
@@
 			)
 		)
-		(property "Value" "RC0402FR-0713K7L"
+		(property "Value" "0402WGF1332TCE"
 			(at 233.934 260.4262 0)
 			(hide yes)
@@
 			)
 		)
-		(property "Description" "RES 13.7K OHM 1% 1/16W 0402"
+		(property "Description" "RES 13.3K OHM 1% 1/16W 0402"
 			(at 232.41 251.2822 0)
 			(hide yes)
@@
 			)
 		)
-		(property "RESISTANCE" "13.7kR"
+		(property "RESISTANCE" "13.3kR"
 			(at 234.95 266.5222 0)
 			(show_name no)
@@
 			)
 		)
-		(property "PLANNED MPN" "RC0402FR-0713K7L"
+		(property "PLANNED MPN" "0402WGF1332TCE"
 			(at 232.41 251.2822 0)
 			(hide yes)
@@
 			)
 		)
-		(property "PLANNED MFR" "Yageo"
+		(property "PLANNED MFR" "UNI-ROYAL"
 			(at 232.41 251.2822 0)
 			(hide yes)
@@
 			)
 		)
-		(property "PLANNED LCSC" "C274888"
+		(property "PLANNED LCSC" "C122547"
 			(at 232.41 251.2822 0)
 			(hide yes)
@@
 			)
 		)
-		(property "PLANNED NOTE" "As specified; in LCSC stock (checked 2026-10-06)"
+		(property "PLANNED NOTE" "13.3k 1% 0402 for 5V buck at 5.11 V (was 13.7k); same UNI-ROYAL range as the 100k (C25741)"
 			(at 232.41 251.2822 0)
 			(hide yes)
@@
 			)
 		)
-		(property "MANUFACTURER" "Yageo"
+		(property "MANUFACTURER" "UNI-ROYAL"
 			(at 232.41 251.2822 0)
 			(hide yes)
@@
 				(path "/30e82bf5-1344-486b-817c-02d3b0649ce4/3c398828-e355-49f6-be37-cb3640d2c671/4eeafcb7-a684-4b4d-adeb-0d10d663bf3a"
 					(reference "R38")
-					(unit 0)
+					(unit 1)
 				)
 			)
