File: experiments/nick_raw_routing/BM_Mote_1_PowerMon.kicad_sch (KiCad schematic)
At the start: 4 parts, among them U4 INA232AIDDFR

Commit message: Added I2C0, I2C1, I2C2 and fix to load switch
Other:
- note added: "I2C0 (Pi GPIO0/1) · Address 0x41 (A0 = GND)"
- note removed: "I2C Address: 0x41"
Changed lines of the file:
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@@
 		(comment 3 "Derived from Sofar Bristlemouth mote 000639-AB")
 	)
-	(text "I2C Address: 0x41"
+	(text "I2C0 (Pi GPIO0/1) · Address 0x41 (A0 = GND)"
 		(exclude_from_sim no)
-		(at 203.2 136.9822 0)
+		(at 175.26 132.08 0)
 		(effects
 			(font
@@
 	(text_box "Power Monitor"
 		(exclude_from_sim no)
-		(at 257.81 191.5922 0)
-		(size -54.61 6.35)
+		(at 203.2 191.5922 0)
+		(size 54.61 6.35)
 		(margins 0.9525 0.9525 0.9525 0.9525)
 		(stroke

Commit message: Fix import connectivity
Connections:
- net P_IN: now also R8.2
- net P_OUT: now also R8.1
Other:
- note added: "I2C0 (Pi GPIO0/1) · Address 0x41 (A0 = VS)"
- note removed: "I2C0 (Pi GPIO0/1) · Address 0x41 (A0 = GND)"

Commit message: updates before the sofar review
Parts:
- R8: ALT NOTE Sofar review: power-path current sense; check land pattern -> (none); ALT1 LCSC C308571 -> (none); ALT1 MFR ROHM -> (none); ALT1 MPN PMR03EZPFU10L0 -> (none); ALT2 LCSC C5334451 -> (none); ALT2 MFR Vishay -> (none); ALT2 MPN WSLP0603R0100FEA -> (none); PLANNED LCSC (none) -> wait for JLC update; SOURCING JLC global sourcing (first build) until an ALT is approved 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 -> JLC global sourcing (first build)
Changed lines of the file:
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@@
 			)
 		)
-		(property "ALT1 MPN" "PMR03EZPFU10L0"
+		(property "ALT1 MPN" ""
 			(at 173.99 156.21 0)
 			(hide yes)
@@
 			)
 		)
-		(property "ALT1 MFR" "ROHM"
+		(property "ALT1 MFR" ""
 			(at 173.99 156.21 0)
 			(hide yes)
@@
 			)
 		)
-		(property "ALT1 LCSC" "C308571"
+		(property "ALT1 LCSC" ""
 			(at 173.99 156.21 0)
 			(hide yes)
@@
 			)
 		)
-		(property "ALT2 MPN" "WSLP0603R0100FEA"
+		(property "ALT2 MPN" ""
 			(at 173.99 156.21 0)
 			(hide yes)
@@
 			)
 		)
-		(property "ALT2 MFR" "Vishay"
+		(property "ALT2 MFR" ""
 			(at 173.99 156.21 0)
 			(hide yes)
@@
 			)
 		)
-		(property "ALT2 LCSC" "C5334451"
+		(property "ALT2 LCSC" ""
 			(at 173.99 156.21 0)
 			(hide yes)
@@
 			)
 		)
-		(property "ALT NOTE" "Sofar review: power-path current sense; check land pattern"
+		(property "ALT NOTE" ""
 			(at 173.99 156.21 0)
 			(hide yes)
@@
 			)
 		)
-		(property "SOURCING" "JLC global sourcing (first build) until an ALT is approved (D26)"
+		(property "SOURCING" "JLC global sourcing (first build) "
 			(at 173.99 156.21 0)
 			(hide yes)
@@
 			)
 		)
-		(property "PLANNED LCSC" ""
+		(property "PLANNED LCSC" "wait for JLC update"
 			(at 173.99 156.21 0)
 			(hide yes)
